File: cad_files/mm6d/mm6d.kicad_pcb (KiCad board)
At the start: 2 copper layers, 0 parts

Commit message: 200723
Other:
- rule pad_to_mask_clearance: 0 -> 0.2
Changed lines of the file:
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@@
     (links 0)
     (no_connects 0)
-    (area 0 0 0 0)
+    (area 143.467767 98.7286 159.86059 111.3786)
     (thickness 1.6)
     (drawings 0)
@@
   (page A4)
   (title_block
-    (company "Pozsar Zsolt")
+    (title "MM6D Remote controlled switching box")
+    (date 2020-06-12)
+    (rev 200612)
+    (company "Pozsar Zsolt - http://www.szerafingomba.hu")
+    (comment 4 "Draw no.: 59/11/3")
   )
   (layers
@@
   (setup
     (last_trace_width 0.25)
+    (user_trace_width 0.5)
+    (user_trace_width 1)
+    (user_trace_width 2.5)
     (trace_clearance 0.2)
     (zone_clearance 0.508)
@@
     (trace_min 0.2)
     (segment_width 0.2)
-    (edge_width 0.1)
+    (edge_width 0.15)
     (via_size 0.6)
     (via_drill 0.4)
@@
     (mod_text_size 1 1)
     (mod_text_width 0.15)
-    (pad_size 1.5 1.5)
-    (pad_drill 0.6)
-    (pad_to_mask_clearance 0)
-    (aux_axis_origin 0 0)
-    (visible_elements FFFFFF7F)
+    (pad_size 1.7272 2.032)
+    (pad_drill 1)
+    (pad_to_mask_clearance 0.2)
+    (aux_axis_origin 20.32 19.05)
+    (visible_elements 7FFEFF7F)
     (pcbplotparams
-      (layerselection 0x00030_80000001)
+      (layerselection 0x01020_00000000)
       (usegerberextensions false)
-      (excludeedgelayer true)
-      (linewidth 0.100000)
-      (plotframeref false)
+      (excludeedgelayer false)
+      (linewidth 0.150000)
+      (plotframeref true)
       (viasonmask false)
       (mode 1)
@@
       (psa4output false)
       (plotreference true)
-      (plotvalue true)
+      (plotvalue false)
       (plotinvisibletext false)
       (padsonsilk false)
       (subtractmaskfromsilk false)
-      (outputformat 1)
+      (outputformat 4)
       (mirror false)
-      (drillshape 1)
+      (drillshape 2)
       (scaleselection 1)
       (outputdirectory ""))
