File: cad_files/mm6d/mm6d.sch (KiCad schematic (older format))
At the start: 55 parts, among them P101 CONN_01X02, P102 CONN_01X02

Commit message: 200723
Parts:
- removed D? (x2): LED-CIRCLE, symbol LED-CIRCLE
- added P?: CONN_01X03, symbol CONN_01X03
- added P?: CONN_01X02, Socket_Strips:Socket_Strip_Straight_1x02, symbol CONN_01X02
- D?: value LED-CIRCLE -> yellow
- D?: value LED-CIRCLE -> red
- D? (x3): value yellow -> green
- gave numbers to parts that had none: 2
Connections:
- wire segments 164 -> 169
- no-connect marks 8 -> 16
Other:
- note added: "Accu"
- note added: "Console"
- note added: "Inputs"
- note added: "Outputs"
- note added: "Piezo\nspeaker"
- note removed: "Piezo speaker"
- moved on the sheet: D101, D?, P101, P102, P?, Q?, R?, U101-JP1, U101-JP3, U?

Commit message: 200723
Parts:
- removed Q? (x8): Q_NPN_BCE, symbol Q_NPN_BCE
- added Q101, Q102, Q103, Q104: BC182, TO_SOT_Packages_THT:TO-92_Inline_Narrow_Oval, symbol Q_NPN_EBC
- added Q105, Q106, Q107, Q108: BD135, TO_SOT_Packages_THT:SOT126_SOT32_Housing_Horizontal, symbol Q_NPN_ECB
- D101, D102, D103, D104: renamed from D?; value diode -> 1N4001; footprint (none) -> Diodes_THT:Diode_DO-41_SOD81_Horizontal_RM10
- D105, D106, D108, D109, D110, D111, D112: renamed from D?; footprint (none) -> LEDs:LED-5MM
- D113: renamed from D?; value diode -> 1N4007; footprint (none) -> TO_SOT_Packages_THT:TO-92_Inline_Narrow_Oval
- D114, D115, D116: renamed from D?; value diode -> 1N4007; footprint (none) -> Diodes_THT:Diode_DO-41_SOD81_Horizontal_RM10
- P101, P106: renamed from P?; footprint (none) -> Socket_Strips:Socket_Strip_Straight_1x05
- P102: renamed from P?; footprint (none) -> Socket_Strips:Socket_Strip_Straight_1x03
- R101, R102, R103, R104: renamed from R?; value R -> 1.5k; footprint (none) -> Discret:R3
- R105, R106, R107, R108: renamed from R?; value R -> 4.7k; footprint (none) -> Discret:R3
- R109, R110, R111, R112, R113: renamed from R?; value R -> 390; footprint (none) -> Discret:R3
- R114, R115, R116, R117: renamed from R?; value R -> 1k; footprint (none) -> Discret:R3
- U101, U102, U103, U104: renamed from U?; footprint DIP-6 -> Housings_DIP:DIP-6_W7.62mm_LongPads
- U101-JP101: renamed from U101-JP1; footprint (none) -> Socket_Strips:Socket_Strip_Straight_1x16
- U101-JP102: renamed from U101-JP3; footprint (none) -> Socket_Strips:Socket_Strip_Straight_1x12
- gave numbers to parts that had none: 1
- renumbered D101 to D107, P101 to P103, P102 to P104

Commit message: 200724
Parts:
- removed D105: yellow, LEDs:LED-5MM, symbol LED-CIRCLE
- removed D106: red, LEDs:LED-5MM, symbol LED-CIRCLE
- D111: renamed from D113; footprint TO_SOT_Packages_THT:TO-92_Inline_Narrow_Oval -> Diodes_THT:Diode_DO-41_SOD81_Horizontal_RM10
- renumbered D107 to D105, D108 to D106, D109 to D107, D110 to D108, D111 to D109, D112 to D110, D114 to D112, D115 to D113, D116 to D114
Connections:
- wire segments 169 -> 165
Other:
- note added: "Activity"
- note added: "General error"
- note added: "Heater on"
- note added: "Lamp on"
- note added: "Ventilator on"
- moved on the sheet: D101, D102, D103, D104, P101, R101, R102, R103, R104

Commit message: 200727
Parts:
- added R118: 1.8k, Discret:R3, symbol R
Connections:
- wire segments 165 -> 166
Changed lines of the file:
@@
 	4600 5350 4000 5350
 Wire Wire Line
-	4600 2650 4600 5350
+	4600 2650 4600 5550
 Wire Wire Line
 	4000 3050 4150 3050
@@
 Wire Wire Line
 	9150 2200 9150 5050
+$Comp
+L R R118
+U 1 1 5F1E719C
+P 4600 5700
+F 0 "R118" V 4725 5675 50  0000 C CNN
+F 1 "1.8k" V 4475 5675 50  0000 C CNN
+F 2 "Discret:R3" V 4530 5700 50  0001 C CNN
+F 3 "" H 4600 5700 50  0000 C CNN
+	1    4600 5700
+	-1   0    0    1
+$EndComp
+Connection ~ 4600 5350
+$Comp
+L pzs_others:0V #PWR?
+U 1 1 5F1E7647
+P 4600 6000
+F 0 "#PWR?" H 4600 5750 50  0001 C CNN
+F 1 "0V" H 4600 5850 50  0001 C CNN
+F 2 "" H 4600 6000 50  0000 C CNN
+F 3 "" H 4600 6000 50  0000 C CNN
+	1    4600 6000
+	1    0    0    -1
+$EndComp
+Wire Wire Line
+	4600 5850 4600 6000
 $EndSCHEMATC

Commit message: 200907
Parts:
- Q105, Q106, Q107, Q108: value BD135 -> BD137
- renumbered U101-JP101 to U105-JP101, U101-JP102 to U105-JP102
Other:
- note added: "U105"
- note removed: "U101"
Changed lines of the file:
@@
 Adafruit\nHuzzah\nFeather
 Text Notes 5625 4875 0    50   ~ 0
-U101
+U105
 Text Notes 5800 1250 0    60   ~ 0
 5V DC
@@
 $EndComp
 $Comp
-L CONN_01X12 U101-JP102
+L CONN_01X12 U105-JP102
 U 1 1 5F19AC49
 P 6150 4200
-F 0 "U101-JP102" H 6150 5300 50  0000 C CNN
+F 0 "U105-JP102" H 6150 5300 50  0000 C CNN
 F 1 "CONN_01X12" V 6250 4200 50  0001 C CNN
 F 2 "Socket_Strips:Socket_Strip_Straight_1x12" H 6150 4200 50  0001 C CNN
@@
 $EndComp
 $Comp
-L CONN_01X16 U101-JP101
+L CONN_01X16 U105-JP101
 U 1 1 5F19AC96
 P 5500 4000
-F 0 "U101-JP101" H 5500 3100 50  0000 C CNN
+F 0 "U105-JP101" H 5500 3100 50  0000 C CNN
 F 1 "CONN_01X16" V 5600 4000 50  0001 C CNN
 F 2 "Socket_Strips:Socket_Strip_Straight_1x16" H 5500 4000 50  0001 C CNN
@@
 U 1 1 5F19E2E1
 P 4150 2500
-F 0 "R105" V 4070 2490 50  0000 C CNN
+F 0 "R105" V 4145 2500 39  0000 C CNN
 F 1 "4.7k" V 4250 2500 50  0000 C CNN
 F 2 "Discret:R3" V 4080 2500 50  0001 C CNN
@@
 U 1 1 5F19E41E
 P 4300 2500
-F 0 "R106" V 4220 2490 50  0000 C CNN
-F 1 "4.7k" V 4300 2070 50  0000 C CNN
+F 0 "R106" V 4295 2500 39  0000 C CNN
+F 1 "4.7k" V 4225 2300 50  0000 C CNN
 F 2 "Discret:R3" V 4230 2500 50  0001 C CNN
 F 3 "" H 4300 2500 50  0000 C CNN
@@
 U 1 1 5F19E4AF
 P 4450 2500
-F 0 "R107" V 4370 2490 50  0000 C CNN
-F 1 "4.7k" V 4450 2070 50  0000 C CNN
+F 0 "R107" V 4445 2500 39  0000 C CNN
+F 1 "4.7k" V 4375 2300 50  0000 C CNN
 F 2 "Discret:R3" V 4380 2500 50  0001 C CNN
 F 3 "" H 4450 2500 50  0000 C CNN
@@
 U 1 1 5F19E543
 P 4600 2500
-F 0 "R108" V 4520 2490 50  0000 C CNN
-F 1 "4.7k" V 4600 2070 50  0000 C CNN
+F 0 "R108" V 4595 2500 39  0000 C CNN
+F 1 "4.7k" V 4475 2500 50  0000 C CNN
 F 2 "Discret:R3" V 4530 2500 50  0001 C CNN
 F 3 "" H 4600 2500 50  0000 C CNN
@@
 P 8550 4650
 F 0 "Q107" H 8750 4700 50  0000 L CNN
-F 1 "BD135" H 8750 4600 50  0000 L CNN
+F 1 "BD137" H 8750 4600 50  0000 L CNN
 F 2 "TO_SOT_Packages_THT:SOT126_SOT32_Housing_Horizontal" H 8750 4750 50  0001 C CNN
 F 3 "" H 8550 4650 50  0000 C CNN
@@
 P 8550 5600
 F 0 "Q108" H 8750 5650 50  0000 L CNN
-F 1 "BD135" H 8750 5550 50  0000 L CNN
+F 1 "BD137" H 8750 5550 50  0000 L CNN
 F 2 "TO_SOT_Packages_THT:SOT126_SOT32_Housing_Horizontal" H 8750 5700 50  0001 C CNN
 F 3 "" H 8550 5600 50  0000 C CNN
@@
 P 8550 3700
 F 0 "Q106" H 8750 3750 50  0000 L CNN
-F 1 "BD135" H 8750 3650 50  0000 L CNN
+F 1 "BD137" H 8750 3650 50  0000 L CNN
 F 2 "TO_SOT_Packages_THT:SOT126_SOT32_Housing_Horizontal" H 8750 3800 50  0001 C CNN
 F 3 "" H 8550 3700 50  0000 C CNN
@@
 P 8550 2750
 F 0 "Q105" H 8750 2800 50  0000 L CNN
-F 1 "BD135" H 8750 2700 50  0000 L CNN
+F 1 "BD137" H 8750 2700 50  0000 L CNN
 F 2 "TO_SOT_Packages_THT:SOT126_SOT32_Housing_Horizontal" H 8750 2850 50  0001 C CNN
 F 3 "" H 8550 2750 50  0000 C CNN

Commit message: 201007
Parts:
- removed D106: blue, LEDs:LED-5MM, symbol LED-CIRCLE
- removed D107, D108, D109: green, LEDs:LED-5MM, symbol LED-CIRCLE
- removed D110: red, LEDs:LED-5MM, symbol LED-CIRCLE
- removed R110, R111, R112, R113: 390, Discret:R3, symbol R
- added C103: 4.7u, symbol device:CP_Small
- added P106: CONN_01X02, Socket_Strips:Socket_Strip_Straight_1x02, symbol CONN_01X02
- added U106: 7805, symbol 7805
- renumbered D111 to D106, D112 to D107, D113 to D108, D114 to D109, P106 to P107, R118 to R109, R109 to R110, R114 to R111, R115 to R112, R116 to R113, R117 to R114
Connections:
- wire segments 166 -> 158
Other:
- note added: "12V DC"
- note added: "Active\n LED"
- note removed: "5V DC"
- note removed: "Activity"
- note removed: "General error"
- note removed: "Heater on"
- note removed: "Lamp on"
- note removed: "Ventilator on"
- moved on the sheet: D101, D102, D103, D104, D105, D106, D107, D108, D109, P101, P103, P107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
