File: cad_files/wiring/wiring.sch (KiCad schematic (older format))
At the start: 62 parts

Commit message: 200725
Parts:
- BT1: renamed from BT?; value Battery -> 3.7V 500mAh; Field4 (none) -> LiPoly accumulator
- C1: renamed from C?; value CP_Small -> 1000u
- C2: renamed from C?; value CP_Small -> 1u Ta
- D1, D7: renamed from D?; value LED-CIRCLE -> white
- D6: renamed from D?; value D -> 1N4007
- LS1: renamed from LS?; value Speaker_Ultrasound -> Piezo speaker
- R1: renamed from R?; value R -> 47k
- R2: renamed from R?; value R -> 1.5k
- gave numbers to parts that had none: 53
Connections:
- wire segments 169 -> 168
Other:
- note added: "Mains (230V AC)\n\nL\n\nN\n\nPE"
- note added: "Manual mode"
- moved on the sheet: AK5, AK6, AK7, BT1, C1, C2, D1, D2, D3, D4, D5, D6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

Commit message: 200725
Parts:
- removed K1a, K2a, K3a, K4a: switch_1P, symbol switch_1P
- added BT2: 9V, symbol Battery
- added D10: yellow, symbol LED-CIRCLE
- added D8, D9: 1N4001, symbol D
- added F2: F0.05A, symbol Fuse
- added K1a, K2a, K3a, K4a, SW4: auxcontalt, symbol auxcontalt
- added P5, P6, P8: screw_conn, symbol screw_conn
- added R3: 1,5k, symbol R
- F3: renamed from F2; value Fuse -> T0.5A
- F4: renamed from F3; value Fuse -> F0.5A
- F5: renamed from F4; value Fuse -> F0.8A
- K1, K2, K3: value electromagnetic_actor_1 -> Finder 40.52; Field4 (none) -> 12V 650mW
- K4: value electromagnetic_actor_1 -> Finder 40.51; Field4 (none) -> 12V 650mW
- Tr1: value transformer_1P_1S -> 230/12V 20VA
- renumbered AK5 to AK1, AK6 to AK2, AK7 to AK3, D8 to D11, F5 to F6, F6 to F7, F7 to F8, P12 to P10, P13 to P11, P14 to P12, P15 to P13, P16 to P14, P17 to P15, P18 to P16, P19 to P17, P20 to P18, J1 to P4, P10 to P7, P11 to P9, R3 to R4
Connections:
- wire segments 168 -> 200
- no-connect marks 0 -> 13
Other:
- note added: "Alarm sensor"
- note added: "C R G"
- note added: "Console"
- note added: "Heater"
- note added: "Lamp"
- note added: "Manual\n mode"
- note added: "Operation\n mode"
- note added: "PE N L"
- note added: "Status lamp"
- note added: "Ventilator"
- moved on the sheet: P7

Commit message: 200725
Connections:
- net +12V: no longer F4.1, K1a.~ (B)
- net GND: no longer P5.1
- net at P101.5 (P5): now also P5.1
- net at AK1.~ (B), AK2.~ (B): no longer AK3.~ (B), R4.2
- net at SW2b.~ (B), SW3b.~ (B): no longer R3.2, SW1b.~ (B)
- new net: AK1.~ (B), AK2.~ (B), AK3.~ (B), R4.2
- new net: F4.1, K1a.~ (B)
- new net: R3.2, SW1b.~ (B), SW2b.~ (B), SW3b.~ (B)
Other:
- moved on the sheet: D10
Changed lines of the file:
@@
 encoding utf-8
 Sheet 1 1
-Title "MM6D Remote controlled switching box"
+Title "MM6D Remote controlled switching device"
 Date "2020-06-12"
 Rev "200612"
@@
 L LED-CIRCLE D10
 U 1 1 5F1C6BFD
-P 5750 5550
-F 0 "D10" H 5750 5700 50  0000 C CNN
-F 1 "yellow" H 5750 5375 50  0000 C CNN
-F 2 "" H 5750 5550 50  0000 C CNN
-F 3 "" H 5750 5550 50  0000 C CNN
-	1    5750 5550
+P 5800 5550
+F 0 "D10" H 5800 5700 50  0000 C CNN
+F 1 "yellow" H 5800 5375 50  0000 C CNN
+F 2 "" H 5800 5550 50  0000 C CNN
+F 3 "" H 5800 5550 50  0000 C CNN
+	1    5800 5550
 	-1   0    0    -1
 $EndComp
@@
 L 0V #PWR10
 U 1 1 5F1C6C03
-P 6025 5650
-F 0 "#PWR10" H 6025 5400 50  0001 C CNN
-F 1 "0V" H 6025 5500 50  0001 C CNN
-F 2 "" H 6025 5650 50  0000 C CNN
-F 3 "" H 6025 5650 50  0000 C CNN
-	1    6025 5650
+P 6075 5650
+F 0 "#PWR10" H 6075 5400 50  0001 C CNN
+F 1 "0V" H 6075 5500 50  0001 C CNN
+F 2 "" H 6075 5650 50  0000 C CNN
+F 3 "" H 6075 5650 50  0000 C CNN
+	1    6075 5650
 	1    0    0    -1
 $EndComp
@@
 L 0V #PWR4
 U 1 1 5F1CF34F
-P 3000 6800
-F 0 "#PWR4" H 3000 6550 50  0001 C CNN
-F 1 "0V" H 3000 6650 50  0001 C CNN
-F 2 "" H 3000 6800 50  0000 C CNN
-F 3 "" H 3000 6800 50  0000 C CNN
-	1    3000 6800
+P 2850 8650
+F 0 "#PWR4" H 2850 8400 50  0001 C CNN
+F 1 "0V" H 2850 8500 50  0001 C CNN
+F 2 "" H 2850 8650 50  0000 C CNN
+F 3 "" H 2850 8650 50  0000 C CNN
+	1    2850 8650
 	0    1    -1   0
 $EndComp
@@
 	7425 5850 7425 3800
 Wire Wire Line
-	3100 6800 3100 6900
-Wire Wire Line
-	3100 6800 3000 6800
+	2950 8650 2950 8750
+Wire Wire Line
+	2950 8650 2850 8650
 Wire Wire Line
 	3300 6750 3300 6900
@@
 	4325 5550 5025 5550
 Wire Wire Line
-	5325 5550 5550 5550
-Wire Wire Line
-	6025 5550 6025 5650
-Wire Wire Line
-	6025 5550 5950 5550
+	5325 5550 5600 5550
+Wire Wire Line
+	6075 5550 6075 5650
+Wire Wire Line
+	6075 5550 6000 5550
 Wire Wire Line
 	5825 6650 5825 6550
 Wire Wire Line
 	5825 6650 6425 6650
-Connection ~ 10875 3100
-Wire Wire Line
-	10875 3200 6225 3200
-Wire Wire Line
-	6225 3200 6225 6650
+Wire Wire Line
+	6225 1100 6225 6650
 Connection ~ 5125 6000
 Wire Wire Line
@@
 Connection ~ 5225 2350
 Wire Wire Line
-	5925 5100 5925 2350
-Wire Wire Line
-	1175 5100 5925 5100
+	5925 2350 5925 5100
+Wire Wire Line
+	5925 5100 1175 5100
 Wire Wire Line
 	1275 5000 1275 5200
@@
 	1275 4200 1275 4300
 Wire Wire Line
-	6125 2400 8575 2400
-Wire Wire Line
-	6125 3600 6125 2400
+	6125 2350 8575 2350
+Wire Wire Line
+	6125 3600 6125 2350
 Wire Wire Line
 	1175 3600 6125 3600
@@
 	7125 5850 7025 5850
 Wire Wire Line
-	5225 825  5225 2150
-Wire Wire Line
-	5225 2150 4075 2150
+	4075 2150 7525 2150
 Wire Wire Line
 	3975 1100 4075 1100
@@
 Connection ~ 3425 1500
 Wire Wire Line
-	3425 1100 3425 1500
-Wire Wire Line
-	3325 1100 3425 1100
+	3425 1500 3425 1100
+Wire Wire Line
+	3425 1100 3325 1100
 Connection ~ 2125 1300
 Wire Wire Line
-	2125 1100 2125 1300
-Wire Wire Line
-	2225 1100 2125 1100
+	2125 1300 2125 1100
+Wire Wire Line
+	2125 1100 2225 1100
 Wire Wire Line
 	1675 2850 2025 2850
@@
 	9325 1300 9325 2600
 Wire Wire Line
-	7525 900  7525 3450
+	7525 2150 7525 3450
 Wire Wire Line
 	8225 3950 8225 3000
@@
 	7025 3400 7025 5200
 Wire Wire Line
-	4900 3400 7025 3400
+	6725 3400 7025 3400
 Wire Wire Line
 	6725 1100 6725 3500
@@
 	10875 3100 10675 3100
 Wire Wire Line
-	10875 1100 10875 3200
-Wire Wire Line
 	4825 1100 10875 1100
 Wire Wire Line
@@
 	9675 2550 9675 2650
 Wire Wire Line
-	5225 900  7525 900
-Wire Wire Line
 	1175 3300 1275 3300
 Wire Wire Line
-	8575 2400 8575 2650
+	8575 2350 8575 2650
 Wire Wire Line
 	10575 2250 10575 2650
@@
 Connection ~ 3625 2950
 Wire Wire Line
-	5925 2350 4975 2350
+	4975 2350 5925 2350
 Wire Wire Line
 	5225 2350 5225 2500
@@
 L +12V #PWR8
 U 1 1 5F1DAD60
-P 5225 825
-F 0 "#PWR8" H 5225 675 50  0001 C CNN
-F 1 "+12V" H 5225 965 50  0000 C CNN
-F 2 "" H 5225 825 50  0000 C CNN
-F 3 "" H 5225 825 50  0000 C CNN
-	1    5225 825
-	1    0    0    -1
-$EndComp
-Connection ~ 5225 900
+P 5975 -75
+F 0 "#PWR8" H 5975 -225 50  0001 C CNN
+F 1 "+12V" H 5975 65  50  0000 C CNN
+F 2 "" H 5975 -75 50  0000 C CNN
+F 3 "" H 5975 -75 50  0000 C CNN
+	1    5975 -75
+	1    0    0    -1
+$EndComp
 Text Notes 7100 6250 0    60   ~ 0
 C   R   G
 Text Notes 7075 6375 0    60   ~ 0
 Status lamp
+Connection ~ 6225 1100
+Wire Wire Line
+	4900 3400 6025 3400
+Wire Wire Line
+	6025 3400 6025 1100
+Connection ~ 6025 1100
+Wire Wire Line
+	10875 1100 10875 3100
+Wire Wire Line
+	3100 6900 3100 3700
+Wire Wire Line
+	3100 3700 1175 3700
 $EndSCHEMATC

Commit message: 200907
Parts:
- removed D2, D3, D4, D5: D, symbol D
- removed F2: F0.05A, symbol Fuse
- removed F5: F0.8A, symbol Fuse
- removed Tr1: 230/12V 20VA, symbol transformer_1P_1S
- added P19: CONN_01X05, symbol CONN_01X05
- F1: value Fuse -> 0.5A
- F2: renamed from F3; value T0.5A -> 0.5A
- F3: renamed from F4; value F0.5A -> 0.5A
- K1, K2, K3: value Finder 40.52 -> Finder 40.51.9.012.0000; Field4 12V 650mW -> (none)
- K4: value Finder 40.51 -> Finder 40.51.9.012.0000; Field4 12V 650mW -> (none)
- renumbered AK1 to AK4, AK2 to AK5, AK3 to AK6, F6 to F4, F7 to F5, F8 to F6, U1 to U2
Connections:
- net GND: now also P19.4 (P4)
- net at D6.1 (K), P11.1, P14.1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: now also P19.2 (P2)
- net at P10.1, P13.1, P16.1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: now also P19.3 (P3)
- net at AK4.~ (B), AK5.~ (B): no longer AK6.~ (B), R4.2
- net at F1.1: now also P19.1 (P1)
- net at C1.1, F2.2, F3.2: now also U2.VI, P19.5 (P5)
- net at SW2b.~ (B), SW3b.~ (B): no longer R3.2, SW1b.~ (B)
- net at D8.1 (K), D9.1 (K): now also P6.1
- new net: AK4.~ (B), AK5.~ (B), AK6.~ (B), R4.2
- new net: R3.2, SW1b.~ (B), SW2b.~ (B), SW3b.~ (B)
Other:
- note added: "230V AC\n12V DC\n 24W"
- note added: "U1"
- moved on the sheet: C1, F1, F2, F3, K1a, U2

Commit message: 201007
Parts:
- removed C1: 1000u, symbol CP_Small
- removed C2: 1u Ta, symbol CP_Small
- removed U2: 7805, symbol 7805
- added D3, D4, D5: green, symbol LED-CIRCLE
- added D8: blue, symbol LED-CIRCLE
- added P106: CONN_01X02, symbol CONN_01X02
- added R3, R4, R5: 1,5k, symbol R
- F5: renamed from F2; value 0.5A -> 1.5A
- renumbered AK4 to AK1, AK5 to AK2, AK6 to AK3, D9 to D10, D8 to D11, D7 to D2, D11 to D6, D10 to D7, D6 to D9, F4 to F1, F5 to F2, F6 to F3, F1 to F4, F3 to F6, K1a to K1a1, K2a to K2a1, K3a to K3a1, K4a to K4a1, P16 to P10, P106 to P107, P17 to P11, P18 to P12, P5 to P13, P6 to P14, P9 to P15, P8 to P16, P7 to P17, P4 to P18, P10 to P4, P11 to P5, P12 to P6, P13 to P7, P14 to P8, P15 to P9, R3 to R6, R4 to R7, SW1a to SW1a1, SW1b to SW1b1, SW2a to SW2a1, SW2b to SW2b1, SW3a to SW3a1, SW3b to SW3b1
Connections:
- net +12V is gone; now on an unnamed net: P107.1 (P1)
- net GND: no longer D7.1 (K)
- net at P101.2 (P2): now also SW1b1.~ (B); no longer SW4.~ (B)
- net at P101.3 (P3): now also SW4.~ (B); no longer SW1b1.~ (B)
- net at P103.2 (P2): now also AK3.~ (B), D11.2 (A), F5.1, K1.1 (-), K2.1 (-), K3.1 (-), K4.1 (-), R2.2, SW3b1.~ (B), SW4.~ (B)
- net at K1.2 (+): now also P107.2 (P2); no longer P107.5 (P5)
- net at AK1.~ (B), AK2.~ (B): no longer AK3.~ (B), R7.2
- net at R7.1: now also D7.2 (A); no longer D6.2 (A)
- net at R6.1: now also AK1.~ (B), AK2.~ (B), AK3.~ (B); no longer D7.2 (A)
- net at SW2b1.~ (B), SW3b1.~ (B): no longer R6.2, SW1b1.~ (B)
- new net: D3.1 (K), K2.2 (+), P107.3 (P3), SW1a1.~ (B)
- new net: D4.1 (K), K3.2 (+), P107.4 (P4), SW2a1.~ (B)
- new net: D5.1 (K), K4.2 (+), P107.5 (P5), SW3a1.~ (B)
- new net: R7.2, SW1b1.~ (B), SW2b1.~ (B), SW3b1.~ (B)
- new net: D6.2 (A), R6.2
- new net: D5.2 (A), R5.1
- new net: D4.2 (A), R4.1
- new net: D3.2 (A), R3.1
- new net: D8.1 (K), P106.1 (P1)
- new net: D8.2 (A), P106.2 (P2)
- now unconnected: SW4.~ (B)
Other:
- note added: "Active"
- note added: "Auxiliary\nvoltage"
- note added: "Heater\non"
- note added: "Lamp\non"
- note added: "Manual\nmode"
- note added: "Protection\nerror"
- note added: "Ventilator\non"
- note added: "front panel"
- note removed: "Auxiliary voltage"
- note removed: "Manual mode"
- note removed: "Protection error"
- moved on the sheet: BT1, BT2, D1, D10, D11, D2, D6, D7, D9, F4, F5, F6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

Commit message: 201007
Parts:
- renumbered P12 to P10, P10 to P12, P6 to P4, P4 to P5, P9 to P7, P7 to P9
Connections:
- net at AK1.~ (B), AK2.~ (B): no longer AK3.~ (B), R6.1
- net at SW2b1.~ (B), SW3b1.~ (B): no longer R7.2, SW1b1.~ (B)
- new net: AK1.~ (B), AK2.~ (B), AK3.~ (B), R6.1
- new net: R7.2, SW1b1.~ (B), SW2b1.~ (B), SW3b1.~ (B)
Changed lines of the file:
@@
 $EndComp
 $Comp
-L screw_conn P12
+L screw_conn P10
 U 1 1 5F1B024C
 P 10425 6100
-F 0 "P12" H 10250 6025 40  0000 L CNN
+F 0 "P10" H 10250 6025 40  0000 L CNN
 F 1 "screw_conn" H 10425 6155 30  0001 C CNN
 F 2 "" H 10425 6100 60  0000 C CNN
@@
 $EndComp
 $Comp
-L screw_conn P9
+L screw_conn P7
 U 1 1 5F1B0433
 P 9325 6100
-F 0 "P9" H 9150 6025 40  0000 L CNN
+F 0 "P7" H 9150 6025 40  0000 L CNN
 F 1 "screw_conn" H 9325 6155 30  0001 C CNN
 F 2 "" H 9325 6100 60  0000 C CNN
@@
 $EndComp
 $Comp
-L screw_conn P6
+L screw_conn P4
 U 1 1 5F1B04A4
 P 8225 6100
-F 0 "P6" H 8050 6050 40  0000 L CNN
+F 0 "P4" H 8050 6050 40  0000 L CNN
 F 1 "screw_conn" H 8225 6155 30  0001 C CNN
 F 2 "" H 8225 6100 60  0000 C CNN
@@
 $EndComp
 $Comp
-L screw_conn P10
+L screw_conn P12
 U 1 1 5F1B1CF4
 P 10025 6100
-F 0 "P10" H 9850 6025 40  0000 L CNN
+F 0 "P12" H 9850 6025 40  0000 L CNN
 F 1 "screw_conn" H 10025 6155 30  0001 C CNN
 F 2 "" H 10025 6100 60  0000 C CNN
@@
 $EndComp
 $Comp
-L screw_conn P7
+L screw_conn P9
 U 1 1 5F1B28DC
 P 8925 6100
-F 0 "P7" H 8750 6025 40  0000 L CNN
+F 0 "P9" H 8750 6025 40  0000 L CNN
 F 1 "screw_conn" H 8925 6155 30  0001 C CNN
 F 2 "" H 8925 6100 60  0000 C CNN
@@
 $EndComp
 $Comp
-L screw_conn P4
+L screw_conn P5
 U 1 1 5F1B2B86
 P 7825 6100
-F 0 "P4" H 7650 6050 40  0000 L CNN
+F 0 "P5" H 7650 6050 40  0000 L CNN
 F 1 "screw_conn" H 7825 6155 30  0001 C CNN
 F 2 "" H 7825 6100 60  0000 C CNN

Commit message: 201008
Parts:
- added D2: red, symbol LED-CIRCLE
- added R2: 1.5k, symbol R
- renumbered D9 to D12, D2 to D3, D3 to D4, D4 to D5, D5 to D6, D6 to D7, D7 to D8, D8 to D9, P5 to P6, R2 to R3, R3 to R4, R4 to R5, R5 to R6, R6 to R7, R7 to R8
Connections:
- net at AK3.~ (B), D11.2 (A), F5.1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: now also R4.2, R5.2, R6.2, R2.2
- net at K1.2 (+), P107.2 (P2): now also D2.1 (K)
- net at P11.1, P19.2 (P2), P2.1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: now also D1.1 (K); no longer D12.1 (K)
- net at D12.2 (A): now also F1.~ (B), F2.~ (B), F3.~ (B), F4.2, P1.1; no longer D1.1 (K)
- net at AK1.~ (B), AK2.~ (B): no longer AK3.~ (B), R7.1
- net at SW2b1.~ (B), SW3b1.~ (B): no longer R8.2, SW1b1.~ (B)
- new net: D12.1 (K), R1.2
- new net: AK1.~ (B), AK2.~ (B), AK3.~ (B), R7.1
- new net: R8.2, SW1b1.~ (B), SW2b1.~ (B), SW3b1.~ (B)
- new net: D2.2 (A), R2.1
Other:
- note added: "Alarm\nError"
- note added: "Mains"
- note removed: "Lamp\non"
- note removed: "Mains voltage"
- moved on the sheet: BT2, D1, D10, D11, D12, D9, P102, P106, P18, R1

Commit message: 201028
Parts:
- removed BT2: 9V, symbol Battery
- removed D1, D3: white, symbol LED-CIRCLE
- removed D10, D11: 1N4001, symbol D
- removed D12: 1N4007, symbol D
- removed D2, D7: red, symbol LED-CIRCLE
- removed D4, D5, D6: green, symbol LED-CIRCLE
- removed D8: yellow, symbol LED-CIRCLE
- removed D9: blue, symbol LED-CIRCLE
- removed P103: CONN_01X02, symbol CONN_01X02
- removed P19: CONN_01X05, symbol CONN_01X05
- removed R1: 47k, symbol R
- removed R2, R3: 1.5k, symbol R
- removed R4, R5, R6, R7, R8: 1,5k, symbol R
- removed SW1a1, SW1b1, SW2a1, SW2b1, SW3a1, SW3b1, SW4: auxcontalt, symbol auxcontalt
- added P201, P? (x2): CONN_01X02, symbol CONN_01X02
- added P202, P203, P208, P209: CONN_01X01, symbol CONN_01X01
- added P204: CONN_01X06, symbol CONN_01X06
- added P205, P206, P207: CONN_01X03, symbol CONN_01X03
- added SW1a?, SW1b?, SW2a?, SW2b?, SW3a?, SW3b?, SW?: auxcontalt, symbol auxcontalt
- added Tr? (x2): transformer_1P_1S, symbol transformer_1P_1S
- BT1: Field4 LiPoly accumulator -> LiPoly accu
- LS1: value Piezo speaker -> Piezo
Connections:
- net GND: now also P207.3 (P3)
- net at P101.2 (P2): now also SW1b?.~ (B)
- net at P101.3 (P3): now also SW?.~ (B)
- net at P107.3 (P3): now also P204.1 (P1); no longer K2.2 (+)
- net at P107.4 (P4): now also P204.3 (P3); no longer K3.2 (+)
- net at P107.5 (P5): now also P204.5 (P5); no longer K4.2 (+)
- net at P11.1, P2.1, P5.1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: now also P205.1 (P1), Tr?.~, Tr?.~
- net at F6.1: no longer K1a1.~ (B)
- net at F6.2: no longer F5.2
- net at F4.1: now also Tr?.~, Tr?.~
- net at P14.1: now also P202.1 (P1)
- net at P106.1 (P1): now also P201.1 (P1)
- net at P106.2 (P2): now also P201.2 (P2)
- new net: AK3.~ (B), K1.1 (-), P107.1 (P1), P206.3 (P3)
- new net: F1.~ (B), F2.~ (B), F3.~ (B), F4.2, P1.1, P205.3 (P3)
- new net: AK1.~ (B), AK2.~ (B), AK3.~ (B), P208.1 (P1)
- new net: K2.1 (-), K3.1 (-), K4.1 (-)
- new net: K2.2 (+), P204.2 (P2)
- new net: K3.2 (+), P204.4 (P4)
- new net: K4.2 (+), P204.6 (P6)
- new net: P207.1 (P1), SW1a?.~ (B), SW2a?.~ (B), SW3a?.~ (B)
- new net: SW1b?.~ (B), SW2b?.~ (B)
- new net: P209.1 (P1), SW1b?.~ (B), SW2b?.~ (B), SW3b?.~ (B)
- new net: SW2b?.~ (B), SW3b?.~ (B)
- new net: P206.2 (P2), SW3b?.~ (B), SW?.~ (B)
- new net: P?.1 (P1), Tr?.~ (x2)
- new net: P?.2 (P2), Tr?.~ (x2)
- now unconnected: F5.1
- no-connect marks 13 -> 14
Other:
- note added: "Display board"
- note added: "Main board"
- note removed: "230V AC\n12V DC\n 24W"
- note removed: "Active"
- note removed: "Alarm\nError"
- note removed: "Auxiliary\nvoltage"
- note removed: "Heater\non"
- note removed: "Mains"
- note removed: "Manual\nmode"
- note removed: "Protection\nerror"
- note removed: "U1"
- note removed: "Ventilator\non"
- note removed: "front panel"
- moved on the sheet: BT1, F4, F5, F6, LS1, P102, P104, P105, P106, P107, P13, P14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
