File: cad_files/wiring/wiring.sch (KiCad schematic (older format))
At the start: 63 parts, among them K1 Finder 40.51.9.012.0000, K1a1 auxcontalt, K2 Finder 40.51.9.012.0000, K2a1 auxcontalt, K3 Finder 40.51.9.012.0000, K3a1 auxcontalt, K4 Finder 40.51.9.012.0000, K4a1 auxcontalt, P1 screw_conn, P10 screw_conn, P101 CONN_01X05, P102 CONN_01X03, P104 CONN_01X02, P105 CONN_01X02, P106 CONN_01X02, P107 CONN_01X05, P11 screw_conn, P12 screw_conn, P13 screw_conn, P14 screw_conn, P15 screw_conn, P16 screw_conn, P17 screw_conn, P18 DB9, P2 screw_conn, P201 CONN_01X02, P202 CONN_01X01, P203 CONN_01X01, P204 CONN_01X06, P205 CONN_01X03, P206 CONN_01X03, P207 CONN_01X03, P208 CONN_01X01, P209 CONN_01X01, P3 screw_conn, P4 screw_conn, P5 screw_conn, P6 screw_conn, P7 screw_conn, P8 screw_conn, P9 screw_conn, SW1a? auxcontalt, SW1b? auxcontalt, SW2a? auxcontalt, SW2b? auxcontalt, SW3a? auxcontalt, SW3b? auxcontalt

Commit message: 201029
Parts:
- added P103: CONN_01X02, symbol CONN_01X02
- F5: value 1.5A -> 0,5A
- Tr1, Tr2: renamed from Tr?; value transformer_1P_1S -> 230V/12V 8VA
- gave numbers to parts that had none: 9
- renumbered K2 to K1, K2a1 to K1a1, K3 to K2, K3a1 to K2a1, K4 to K3, K4a1 to K3a1, K1 to K4, K1a1 to K4a1, P101 to P104, P107 to P105, P102 to P106, P104 to P107, P105 to P108, P106 to P109
Connections:
- net GND: now also P103.1 (P1)
- net at AK3.~ (B), K4.1 (-), P105.1 (P1)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: now also F6.1
- net at K4.2 (+), P105.2 (P2): now also P203.1 (P1)
- net at P105.3 (P3), P204.1 (P1): now also K1.2 (+)
- net at P105.4 (P4), P204.3 (P3): now also K2.2 (+)
- net at P105.5 (P5), P204.5 (P5): now also K3.2 (+)
- net at F6.2: now also F5.2, P103.2 (P2)
- net at F5.1: now also K4a1.~ (B)
- net at P204.2 (P2): now also SW1.~ (B); no longer K1.2 (+)
- net at P204.4 (P4): now also SW2.~ (B); no longer K2.2 (+)
- net at P204.6 (P6): now also SW3.~ (B); no longer K3.2 (+)
- net at K4a1.~ (B): now also P16.1
- net at SW'1.~ (B): now also P104.2 (P2); no longer SW'2.~ (B)
- net at SW4.~ (B): now also P104.3 (P3)
- new net: AK1.~ (B), AK2.~ (B), AK3.~ (B), P208.1 (P1)
- new net: F4.1, Tr1.~, Tr2.~
- new net: P207.1 (P1), SW1.~ (B), SW2.~ (B), SW3.~ (B)
- new net: SW'1.~ (B), SW'2.~ (B)
- new net: P209.1 (P1), SW'1.~ (B), SW'2.~ (B), SW'3.~ (B)
- no-connect marks 14 -> 16
Other:
- note added: "12V"
- note added: "230V"
- note added: "8V"
- moved on the sheet: F5, F6, P106, P13, P14, P18

Commit message: 201226
Parts:
- F4: value 0.5A -> 0.25A
- F5: value 0,5A -> 0,8A
- F6: value 0.5A -> 0.8A
- renumbered P104 to P101, P103 to P102, P101 to P103, P102 to P104, P106 to P105, P107 to P106, P108 to P107, P109 to P108, P105 to P109
Connections:
- net at SW1.~ (B): now also P204.2 (P2)
- net at SW'1.~ (B): now also P101.3 (P3); no longer SW'2.~ (B)
- net at P101.2 (P2): now also SW4.~ (B); no longer SW'1.~ (B)
- net at SW2.~ (B): now also P204.4 (P4)
- net at SW3.~ (B): now also P204.6 (P6)
- new net: AK1.~ (B), AK2.~ (B), AK3.~ (B), P208.1 (P1)
- new net: F4.1, Tr1.~, Tr2.~
- new net: P207.1 (P1), SW1.~ (B), SW2.~ (B), SW3.~ (B)
- new net: SW'1.~ (B), SW'2.~ (B)
- new net: P209.1 (P1), SW'1.~ (B), SW'2.~ (B), SW'3.~ (B)
Other:
- note added: "Lamp Ventilator Heater"
- note added: "Manual operation mode"
- note removed: "Manual\n mode"
Changed lines of the file:
@@
 $EndDescr
 $Comp
-L CONN_01X02 P107
+L CONN_01X02 P106
 U 1 1 5F1AEA68
 P 2600 4925
-F 0 "P107" V 2700 4925 50  0000 C CNN
+F 0 "P106" V 2700 4925 50  0000 C CNN
 F 1 "CONN_01X02" V 2700 4925 50  0001 C CNN
 F 2 "" H 2600 4925 50  0000 C CNN
@@
 $EndComp
 $Comp
-L CONN_01X02 P108
+L CONN_01X02 P107
 U 1 1 5F1AEAED
 P 2600 4525
-F 0 "P108" V 2700 4525 50  0000 C CNN
+F 0 "P107" V 2700 4525 50  0000 C CNN
 F 1 "CONN_01X02" V 2700 4525 50  0001 C CNN
 F 2 "" H 2600 4525 50  0000 C CNN
@@
 $EndComp
 $Comp
-L CONN_01X03 P106
+L CONN_01X03 P105
 U 1 1 5F1AEB30
 P 1850 5925
-F 0 "P106" V 1950 5925 50  0000 C CNN
+F 0 "P105" V 1950 5925 50  0000 C CNN
 F 1 "CONN_01X03" V 1950 5925 50  0001 C CNN
 F 2 "" H 1850 5925 50  0000 C CNN
@@
 $EndComp
 $Comp
-L CONN_01X05 P105
+L CONN_01X05 P109
 U 1 1 5F1AEB6F
 P 2600 5500
-F 0 "P105" V 2700 5500 50  0000 C CNN
+F 0 "P109" V 2700 5500 50  0000 C CNN
 F 1 "CONN_01X05" V 2700 5500 50  0001 C CNN
 F 2 "" H 2600 5500 50  0000 C CNN
@@
 P 2200 2350
 F 0 "F6" V 2275 2275 50  0000 C CNN
-F 1 "0.5A" V 2275 2450 50  0000 C CNN
+F 1 "0.8A" V 2275 2450 50  0000 C CNN
 F 2 "" V 2130 2350 50  0000 C CNN
 F 3 "" H 2200 2350 50  0000 C CNN
@@
 P 2200 2150
 F 0 "F5" V 2275 2075 50  0000 C CNN
-F 1 "0,5A" V 2275 2250 50  0000 C CNN
+F 1 "0,8A" V 2275 2250 50  0000 C CNN
 F 2 "" V 2130 2150 50  0000 C CNN
 F 3 "" H 2200 2150 50  0000 C CNN
@@
 P 4275 2800
 F 0 "F4" V 4350 2800 50  0000 C CNN
-F 1 "0.5A" V 4175 2800 50  0000 C CNN
+F 1 "0.25A" V 4175 2800 50  0000 C CNN
 F 2 "" V 4205 2800 50  0000 C CNN
 F 3 "" H 4275 2800 50  0000 C CNN
@@
 F 2 "" V 3475 4635 50  0000 C CNN
 F 3 "" V 3475 4635 50  0000 C CNN
-F 4 "LiPoly accu" V 3325 4575 50  0000 C CNN "Field4"
+F 4 "LiPoly accu" V 3775 4550 50  0000 C CNN "Field4"
 	1    3475 4575
 	0    -1   -1   0
@@
 Status lamp
 $Comp
-L CONN_01X02 P109
+L CONN_01X02 P108
 U 1 1 5F81A1FB
 P 2600 4000
-F 0 "P109" V 2700 4000 50  0000 C CNN
+F 0 "P108" V 2700 4000 50  0000 C CNN
 F 1 "CONN_01X02" V 2700 4000 50  0001 C CNN
 F 2 "" H 2600 4000 50  0000 C CNN
@@
 	0    -1   -1   0
 $EndComp
-Text Notes 3950 6125 0    60   ~ 0
-Manual\n mode
+Text Notes 3925 7525 0    60   ~ 0
+Manual operation mode
 $Comp
 L auxcontalt SW4
@@
 $EndComp
 $Comp
-L CONN_01X02 P102
+L CONN_01X02 P104
 U 1 1 5F9A3518
 P 2600 3150
-F 0 "P102" V 2700 3150 50  0000 C CNN
+F 0 "P104" V 2700 3150 50  0000 C CNN
 F 1 "CONN_01X02" V 2700 3150 50  0001 C CNN
 F 2 "" H 2600 3150 50  0000 C CNN
@@
 $EndComp
 $Comp
-L CONN_01X02 P101
+L CONN_01X02 P103
 U 1 1 5F9A38F0
 P 2600 3400
-F 0 "P101" V 2700 3400 50  0000 C CNN
+F 0 "P103" V 2700 3400 50  0000 C CNN
 F 1 "CONN_01X02" V 2700 3400 50  0001 C CNN
 F 2 "" H 2600 3400 50  0000 C CNN
@@
 Display board
 $Comp
-L CONN_01X05 P104
+L CONN_01X05 P101
 U 1 1 5F9BE00B
 P 2600 6175
-F 0 "P104" V 2700 6200 50  0000 C CNN
+F 0 "P101" V 2700 6200 50  0000 C CNN
 F 1 "CONN_01X05" V 2700 6175 50  0001 C CNN
 F 2 "" H 2600 6175 50  0000 C CNN
@@
 	6350 4500 6350 5500
 Wire Wire Line
-	6250 3900 6250 5800
+	6250 5800 6250 3900
 Wire Wire Line
 	6250 3900 6725 3900
@@
 	6050 6975 6050 6875
 Connection ~ 5800 6975
-Wire Wire Line
-	5950 6175 5950 6525
 Wire Wire Line
 	5800 5900 5800 6975
@@
 	1550 5825 1650 5825
 Wire Wire Line
-	2800 6075 3750 6075
-Wire Wire Line
-	3750 6075 3750 6525
-Wire Wire Line
-	2800 6175 5950 6175
+	2800 6175 3750 6175
+Wire Wire Line
+	2800 6075 5950 6075
 Wire Wire Line
 	2800 6275 3100 6275
@@
 	2000 3025 2450 3025
 $Comp
-L CONN_01X02 P103
+L CONN_01X02 P102
 U 1 1 5F9AF9FB
 P 1850 3150
-F 0 "P103" V 1950 3150 50  0000 C CNN
+F 0 "P102" V 1950 3150 50  0000 C CNN
 F 1 "CONN_01X02" V 1950 3150 50  0001 C CNN
 F 2 "" H 1850 3150 50  0000 C CNN
@@
 	5225 6000 5225 5225
 Wire Wire Line
-	5425 5225 5425 6075
-Wire Wire Line
-	5425 6075 5150 6075
-Wire Wire Line
-	5150 6075 5150 6525
+	5425 5225 5425 6175
+Wire Wire Line
+	5425 6175 5150 6175
+Wire Wire Line
+	5150 6175 5150 6525
 Wire Wire Line
 	4225 5225 4225 5800
@@
 NoConn ~ 5025 4275
 NoConn ~ 4700 4275
+Wire Wire Line
+	3750 6175 3750 6525
+Wire Wire Line
+	5950 6075 5950 6525
+Text Notes 3550 7350 0    60   ~ 0
+Lamp          Ventilator          Heater
 $EndSCHEMATC

Commit message: 201227
Connections:
- net at AK3.~ (B), F6.1, K4.1 (-)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: now also K1.1 (-), K2.1 (-), K3.1 (-)
- net at SW1.~ (B): now also P204.2 (P2)
- net at SW'1.~ (B): now also P101.3 (P3); no longer SW'2.~ (B)
- net at SW2.~ (B): now also P204.4 (P4)
- net at SW3.~ (B): now also P204.6 (P6)
- net at SW4.~ (B): now also P101.2 (P2)
- new net: AK1.~ (B), AK2.~ (B), AK3.~ (B), P208.1 (P1)
- new net: F4.1, Tr1.~, Tr2.~
- new net: P207.1 (P1), SW1.~ (B), SW2.~ (B), SW3.~ (B)
- new net: SW'1.~ (B), SW'2.~ (B)
- new net: P209.1 (P1), SW'1.~ (B), SW'2.~ (B), SW'3.~ (B)
Changed lines of the file:
@@
 	8375 2250 8375 2650
 Wire Wire Line
-	5875 2250 10575 2250
+	5875 2250 8375 2250
+Wire Wire Line
+	8375 2250 9475 2250
+Wire Wire Line
+	9475 2250 10575 2250
 Wire Wire Line
 	10575 2250 10575 2650
@@
 	9575 3000 9575 3100
 Wire Wire Line
-	2525 1100 10875 1100
+	2525 1100 5225 1100
+Wire Wire Line
+	5225 1100 6725 1100
+Wire Wire Line
+	6725 1100 10875 1100
 Wire Wire Line
 	10875 3100 10675 3100
@@
 	6725 4100 6725 4000
 Wire Wire Line
-	6725 1100 6725 3500
-Wire Wire Line
-	7025 3400 7025 5200
+	6725 1100 6725 3400
+Wire Wire Line
+	6725 3400 6725 3500
+Wire Wire Line
+	7025 3400 7025 4000
+Wire Wire Line
+	7025 4000 7025 4600
+Wire Wire Line
+	7025 4600 7025 5200
 Wire Wire Line
 	7025 5200 6725 5200
@@
 	10225 1500 10225 5950
 Wire Wire Line
-	1125 1700 10025 1700
-Wire Wire Line
-	1125 1500 10225 1500
+	1125 1700 7825 1700
+Wire Wire Line
+	7825 1700 8925 1700
+Wire Wire Line
+	8925 1700 10025 1700
+Wire Wire Line
+	1125 1500 3925 1500
+Wire Wire Line
+	3925 1500 5450 1500
+Wire Wire Line
+	5450 1500 8025 1500
+Wire Wire Line
+	8025 1500 9125 1500
+Wire Wire Line
+	9125 1500 10225 1500
 Wire Wire Line
 	10425 5650 10425 5950
@@
 	8225 1300 8225 2600
 Wire Wire Line
-	1125 1300 10425 1300
+	1125 1300 4525 1300
+Wire Wire Line
+	4525 1300 5650 1300
+Wire Wire Line
+	5650 1300 8225 1300
+Wire Wire Line
+	8225 1300 9325 1300
+Wire Wire Line
+	9325 1300 10425 1300
 Wire Wire Line
 	10425 1300 10425 2600
@@
 	6250 3900 6725 3900
 Wire Wire Line
-	3200 6975 5050 6975
+	3200 6975 3450 6975
+Wire Wire Line
+	3450 6975 4250 6975
+Wire Wire Line
+	4250 6975 5050 6975
 Wire Wire Line
 	4250 6975 4250 6875
@@
 	5550 6325 5550 6525
 Wire Wire Line
-	3950 6325 5650 6325
+	3950 6325 4750 6325
+Wire Wire Line
+	4750 6325 5550 6325
+Wire Wire Line
+	5550 6325 5650 6325
 Wire Wire Line
 	4750 6325 4750 6525
@@
 Connection ~ 4750 6325
 Wire Wire Line
-	5450 6975 6050 6975
+	5450 6975 5800 6975
+Wire Wire Line
+	5800 6975 6050 6975
 Wire Wire Line
 	5450 6975 5450 6875
@@
 	3925 3350 3825 3350
 Wire Wire Line
-	3925 1500 3925 3350
+	3925 1500 3925 3200
+Wire Wire Line
+	3925 3200 3925 3350
 Wire Wire Line
 	3925 3200 3825 3200
 Connection ~ 3925 3200
 Wire Wire Line
-	3825 2800 4125 2800
+	3825 2800 4025 2800
+Wire Wire Line
+	4025 2800 4125 2800
 Wire Wire Line
 	4025 2800 4025 3750
@@
 	4525 2800 4525 1300
 Wire Wire Line
-	6350 5500 2800 5500
-Wire Wire Line
-	2800 5600 6450 5600
-Wire Wire Line
-	2800 5700 6725 5700
+	6350 5500 4925 5500
+Wire Wire Line
+	4925 5500 2800 5500
+Wire Wire Line
+	2800 5600 5125 5600
+Wire Wire Line
+	5125 5600 6450 5600
+Wire Wire Line
+	2800 5700 5325 5700
+Wire Wire Line
+	5325 5700 6725 5700
 Wire Wire Line
 	5325 5700 5325 5225
@@
 	2900 5400 2900 5800
 Wire Wire Line
-	2900 5800 6250 5800
+	2900 5800 4225 5800
+Wire Wire Line
+	4225 5800 6250 5800
 Wire Wire Line
 	5650 4275 5650 1300
@@
 	1550 3100 1650 3100
 Wire Wire Line
-	1550 2150 1550 3100
+	1550 2150 1550 2350
+Wire Wire Line
+	1550 2350 1550 3100
 Wire Wire Line
 	1550 2350 2050 2350
@@
 Text Notes 3550 7350 0    60   ~ 0
 Lamp          Ventilator          Heater
+Wire Wire Line
+	7025 3400 6725 3400
 $EndSCHEMATC

Commit message: 240423
Parts:
- added R201: 15k, symbol Device:R
- AK1, AK2, AK3, K1a1, K2a1, K3a1, K4a1, SW'1, SW'2, SW'3, SW1, SW2, SW3, SW4: symbol auxcontalt -> pzs_others:auxcontalt
- BT1: symbol Battery -> wiring-rescue:Battery
- F1, F2, F3: symbol overcurrent_breaker -> pzs_others:overcurrent_breaker
- F4, F5, F6: symbol Fuse -> wiring-rescue:Fuse
- K1, K2, K3, K4: symbol electromagnetic_actor_1 -> pzs_others:electromagnetic_actor_1
- LS1: symbol Speaker_Ultrasound -> wiring-rescue:Speaker_Ultrasound
- P1, P10, P11, P12, P13, P14, P15, P16, P17, P2, P3, P4, P5, P6, P7, P8, P9: symbol screw_conn -> pzs_others:screw_conn
- P101, P109: symbol CONN_01X05 -> wiring-rescue:CONN_01X05
- P102, P103, P104, P106, P107, P108, P201: symbol CONN_01X02 -> wiring-rescue:CONN_01X02
- P105, P205, P206, P207: symbol CONN_01X03 -> wiring-rescue:CONN_01X03
- P18: symbol DB9 -> wiring-rescue:DB9
- P202, P203, P208, P209: symbol CONN_01X01 -> wiring-rescue:CONN_01X01
- P204: symbol CONN_01X06 -> wiring-rescue:CONN_01X06
- Tr1, Tr2: symbol transformer_1P_1S -> pzs_others:transformer_1P_1S
Connections:
- net at P13.1: now also P101.2 (P2); no longer P101.5 (P5)
- net at SW1.~ (B): now also P204.2 (P2)
- net at SW'1.~ (B): now also P101.3 (P3); no longer SW'2.~ (B)
- net at SW2.~ (B): now also P204.4 (P4)
- net at SW3.~ (B): now also P204.6 (P6)
- net at P206.2 (P2), SW'3.~ (B), SW4.~ (B): now also R201.1
- net at SW4.~ (B): now also R201.2
- new net: AK1.~ (B), AK2.~ (B), AK3.~ (B), P208.1 (P1)
- new net: F4.1, Tr1.~, Tr2.~
- new net: P207.1 (P1), SW1.~ (B), SW2.~ (B), SW3.~ (B)
- new net: SW'1.~ (B), SW'2.~ (B)
- new net: P209.1 (P1), SW'1.~ (B), SW'2.~ (B), SW'3.~ (B)
- new net: P101.5 (P5), SW4.~ (B)
- no-connect marks 16 -> 15
Other:
- note added: "RS-232 TTL"
- note removed: "Console"
