File: cad_files/mainboard/mainboard.kicad_pcb (KiCad board)
At the start: 2 copper layers, 0 parts

Commit message: 201029
Other:
- rule pad_to_mask_clearance: 0.2 -> 0
Changed lines of the file:
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@@
     (links 0)
     (no_connects 0)
-    (area 143.467767 98.7286 159.86059 111.3786)
+    (area 0 0 0 0)
     (thickness 1.6)
     (drawings 0)
@@
     (rev 200612)
     (company "Pozsar Zsolt - http://www.szerafingomba.hu")
+    (comment 1 "Main board")
     (comment 4 "Draw no.: 59/11/3")
   )
@@
   (setup
     (last_trace_width 0.25)
-    (user_trace_width 0.5)
-    (user_trace_width 1)
-    (user_trace_width 2.5)
     (trace_clearance 0.2)
     (zone_clearance 0.508)
@@
     (trace_min 0.2)
     (segment_width 0.2)
-    (edge_width 0.15)
+    (edge_width 0.1)
     (via_size 0.6)
     (via_drill 0.4)
@@
     (mod_text_size 1 1)
     (mod_text_width 0.15)
-    (pad_size 1.7272 2.032)
-    (pad_drill 1)
-    (pad_to_mask_clearance 0.2)
-    (aux_axis_origin 20.32 19.05)
-    (visible_elements 7FFEFF7F)
+    (pad_size 1.5 1.5)
+    (pad_drill 0.6)
+    (pad_to_mask_clearance 0)
+    (aux_axis_origin 0 0)
+    (visible_elements FFFFFF7F)
     (pcbplotparams
-      (layerselection 0x01020_00000000)
+      (layerselection 0x00030_80000001)
       (usegerberextensions false)
-      (excludeedgelayer false)
-      (linewidth 0.150000)
-      (plotframeref true)
+      (excludeedgelayer true)
+      (linewidth 0.100000)
+      (plotframeref false)
       (viasonmask false)
       (mode 1)
@@
       (psa4output false)
       (plotreference true)
-      (plotvalue false)
+      (plotvalue true)
       (plotinvisibletext false)
       (padsonsilk false)
       (subtractmaskfromsilk false)
-      (outputformat 4)
+      (outputformat 1)
       (mirror false)
-      (drillshape 2)
+      (drillshape 1)
       (scaleselection 1)
       (outputdirectory ""))

Commit message: 201030
Parts:
- added C101: 470u, Capacitors_THT:C_Radial_D8_L11.5_P3.5, F.Cu at (153.7, 80.0)
- added C102: 470u, Capacitors_THT:C_Radial_D8_L11.5_P3.5, F.Cu at (153.7, 91.4)
- added C103: 4.7u, Capacitors_THT:C_Rect_L7_W4.5_P5, F.Cu at (167.6, 81.3)
- added C104: 2.2u, Capacitors_THT:C_Rect_L7_W4.5_P5, F.Cu at (167.6, 90.2)
- added D101: 1N4001, Diodes_THT:Diode_DO-41_SOD81_Horizontal_RM10, F.Cu at (137.2, 114.3)
- added D102: 1N4001, Diodes_THT:Diode_DO-41_SOD81_Horizontal_RM10, F.Cu at (137.2, 119.4)
- added D103: 1N4001, Diodes_THT:Diode_DO-41_SOD81_Horizontal_RM10, F.Cu at (137.2, 124.5)
- added D104: 1N4001, Diodes_THT:Diode_DO-41_SOD81_Horizontal_RM10, F.Cu at (137.2, 129.5)
- added D105: 1N4001, Diodes_THT:Diode_DO-41_SOD81_Horizontal_RM10, F.Cu at (137.2, 134.6)
- added D106: 1N4001, Diodes_THT:Diode_DO-41_SOD81_Horizontal_RM10, F.Cu at (137.2, 139.7)
- added D107: 1N4001, Diodes_THT:Diode_DO-41_SOD81_Horizontal_RM10, F.Cu at (137.2, 144.8)
- added D108: 1N4001, Diodes_THT:Diode_DO-41_SOD81_Horizontal_RM10, F.Cu at (137.2, 149.9)
- added D109: 1N4001, Diodes_THT:Diode_DO-41_SOD81_Horizontal_RM10, F.Cu at (85.1, 95.2)
- added D110: 1N4001, Diodes_THT:Diode_DO-41_SOD81_Horizontal_RM10, F.Cu at (85.1, 100.3)
- added D111: 1N4001, Diodes_THT:Diode_DO-41_SOD81_Horizontal_RM10, F.Cu at (85.1, 106.7)
- added D112: 1N4001, Diodes_THT:Diode_DO-41_SOD81_Horizontal_RM10, F.Cu at (85.1, 113.0)
- added D113: 1N4007, Diodes_THT:Diode_DO-41_SOD81_Horizontal_RM10, F.Cu at (232.4, 100.3)
- added D114: 1N4007, Diodes_THT:Diode_DO-41_SOD81_Horizontal_RM10, F.Cu at (243.8, 105.4)
- added D115: 1N4007, Diodes_THT:Diode_DO-41_SOD81_Horizontal_RM10, F.Cu at (255.3, 100.3)
- added D116: 1N4007, Diodes_THT:Diode_DO-41_SOD81_Horizontal_RM10, F.Cu at (266.7, 104.1)
- added P101: CONN_01X05, Socket_Strips:Socket_Strip_Straight_1x05, F.Cu at (191.8, 82.5)
- added P102: CONN_01X02, Socket_Strips:Socket_Strip_Straight_1x02, F.Cu at (198.1, 90.2)
- added P103: CONN_01X02, Socket_Strips:Socket_Strip_Straight_1x02, F.Cu at (198.1, 96.5)
- added P104: CONN_01X02, Socket_Strips:Socket_Strip_Straight_1x02, F.Cu at (198.1, 102.9)
- added P105: CONN_01X03, Socket_Strips:Socket_Strip_Straight_1x03, F.Cu at (208.3, 85.1)
- added P106: CONN_01X02, Socket_Strips:Socket_Strip_Straight_1x02, F.Cu at (209.6, 90.2)
- added P107: CONN_01X02, Socket_Strips:Socket_Strip_Straight_1x02, F.Cu at (208.3, 96.5)
- added P108: CONN_01X02, Socket_Strips:Socket_Strip_Straight_1x02, F.Cu at (208.3, 102.9)
- added P109: CONN_01X05, Socket_Strips:Socket_Strip_Straight_1x05, F.Cu at (198.1, 110.5)
- added Q101: BC182, TO_SOT_Packages_THT:TO-92_Inline_Narrow_Oval, F.Cu at (233.7, 114.3)
- added Q102: BC182, TO_SOT_Packages_THT:TO-92_Inline_Narrow_Oval, F.Cu at (247.7, 115.6)
- added Q103: BC182, TO_SOT_Packages_THT:TO-92_Inline_Narrow_Oval, F.Cu at (257.8, 115.6)
- added Q104: BC182, TO_SOT_Packages_THT:TO-92_Inline_Narrow_Oval, F.Cu at (268.0, 115.6)
- added Q105: BD137, TO_SOT_Packages_THT:SOT126_SOT32_Housing_Horizontal, F.Cu at (237.5, 91.4)
- added Q106: BD137, TO_SOT_Packages_THT:SOT126_SOT32_Housing_Horizontal, F.Cu at (248.9, 91.4)
- added Q107: BD137, TO_SOT_Packages_THT:SOT126_SOT32_Housing_Horizontal, F.Cu at (260.4, 91.4)
- added Q108: BD137, TO_SOT_Packages_THT:SOT126_SOT32_Housing_Horizontal, F.Cu at (271.8, 91.4)
- added R101: 1.5k, Discret:R3, F.Cu at (116.8, 97.8)
- added R102: 1.5k, Discret:R3, F.Cu at (116.8, 100.3)
- added R103: 1.5k, Discret:R3, F.Cu at (116.8, 102.9)
- added R104: 1.5k, Discret:R3, F.Cu at (116.8, 105.4)
- added R105: 4.7k, Discret:R3, F.Cu at (185.4, 88.9)
- added R106: 4.7k, Discret:R3, F.Cu at (185.4, 91.4)
- added R107: 4.7k, Discret:R3, F.Cu at (185.4, 94.0)
- added R108: 4.7k, Discret:R3, F.Cu at (185.4, 96.5)
- added R109: 1.8k, Discret:R3, F.Cu at (185.4, 99.1)
- added R110: 390, Discret:R3, F.Cu at (185.4, 101.6)
- added R111: 1k, Discret:R3, F.Cu at (213.4, 118.1)
- added R112: 1k, Discret:R3, F.Cu at (213.4, 120.7)
- added R113: 1k, Discret:R3, F.Cu at (213.4, 123.2)
- added R114: 1k, Discret:R3, F.Cu at (213.4, 125.7)
- added U101: 7805, TO_SOT_Packages_THT:TO-220_Neutral123_Horizontal_LargePads, F.Cu at (141.0, 99.1)
- added U102: 4N25, Housings_DIP:DIP-6_W7.62mm_LongPads, F.Cu at (109.2, 134.6)
- added U103: 4N25, Housings_DIP:DIP-6_W7.62mm_LongPads, F.Cu at (120.7, 121.9)
- added U104: 4N25, Housings_DIP:DIP-6_W7.62mm_LongPads, F.Cu at (120.7, 134.6)
- added U105: 4N25, Housings_DIP:DIP-6_W7.62mm_LongPads, F.Cu at (109.2, 121.9)
- added U105-JP101: CONN_01X16, Socket_Strips:Socket_Strip_Straight_1x16, F.Cu at (167.6, 138.4)
- added U105-JP102: CONN_01X12, Socket_Strips:Socket_Strip_Straight_1x12, F.Cu at (167.6, 128.3)

Commit message: 201030
Parts:
- added REF**: MountingHole_3.2mm_M3_Pad, Mounting_Holes:MountingHole_3.2mm_M3_Pad, F.Cu at (271.3, 82.3)
- added REF**: MountingHole_3.2mm_M3_Pad, Mounting_Holes:MountingHole_3.2mm_M3_Pad, F.Cu at (271.3, 135.1)
- added REF**: MountingHole_3.2mm_M3_Pad, Mounting_Holes:MountingHole_3.2mm_M3_Pad, F.Cu at (149.4, 82.3)
- added REF**: MountingHole_3.2mm_M3_Pad, Mounting_Holes:MountingHole_3.2mm_M3_Pad, F.Cu at (149.4, 135.1)
- moved U102 131.2 mm to (130.0, 5.08)
- moved U103 131.2 mm to (141.5, -7.62)
- moved U104 131.2 mm to (141.5, 5.08)
- moved U105 131.2 mm to (130.0, -7.62)
- moved D109 128.2 mm to (200.9, 40.4)
- moved D110 128.2 mm to (200.9, 45.5)
- moved D111 128.2 mm to (200.9, 51.8)
- moved D112 128.2 mm to (200.9, 58.2)
- moved P101 93.4 mm to (173.0, -8.89)
- moved P106 93.4 mm to (190.8, -1.27)
- moved R105 93.4 mm to (166.6, -2.54)
- moved U105-JP102 93.4 mm to (148.8, 36.8)
- moved P105 93.4 mm to (189.5, -6.35)
- moved P107 93.4 mm to (189.5, 5.08)
- moved P108 93.4 mm to (189.5, 11.4)
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Routing:
- net GND: track 0.00 -> 58.7 mm
- net Net-(D113-Pad1): track 0.00 -> 57.3 mm
- net Net-(D114-Pad2): track 0.00 -> 40.6 mm
- net Net-(D115-Pad2): track 0.00 -> 35.9 mm
- net Net-(D113-Pad2): track 0.00 -> 28.1 mm
- net Net-(C101-Pad1): track 0.00 -> 27.6 mm
- net Net-(D116-Pad2): track 0.00 -> 24.3 mm
- net Net-(Q104-Pad2): track 0.00 -> 20.6 mm
- net Net-(Q101-Pad2): track 0.00 -> 20.5 mm
- net Net-(C102-Pad1): track 0.00 -> 14.5 mm
- net Net-(D107-Pad2): track 0.00 -> 10.8 mm
- net Net-(D103-Pad2): track 0.00 -> 10.6 mm
- net Net-(D105-Pad2): track 0.00 -> 10.6 mm
- net Net-(D101-Pad2): track 0.00 -> 10.3 mm
- net Net-(Q102-Pad2): track 0.00 -> 9.83 mm
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Other:
- board outline added: 132.1 x 63 mm

Commit message: 201031
Parts:
- moved P101 285.2 mm to (388.0, 178.4), turned to 180 degrees
- moved R101 284.2 mm to (385.5, 169.5), turned to 270 degrees
- moved R102 280.7 mm to (383.0, 169.5), turned to 270 degrees
- moved R103 277.2 mm to (380.4, 169.5), turned to 270 degrees
- moved R104 273.7 mm to (377.9, 169.5), turned to 270 degrees
- moved R105 234.0 mm to (353.8, 137.9)
- moved R106 234.0 mm to (353.8, 140.5)
- moved R107 234.0 mm to (353.8, 143.0)
- moved R108 234.0 mm to (353.8, 145.5)
- moved R109 234.0 mm to (353.8, 148.1)
- moved R110 234.0 mm to (353.8, 150.6)
- moved U105-JP102 226.3 mm to (367.9, 93.8), turned to 90 degrees
- moved U102 218.9 mm to (317.0, 118.9)
- moved U103 206.9 mm to (319.8, 97.2)
- moved U105-JP101 205.7 mm to (348.7, 95.5), turned to 90 degrees
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Routing:
- net GND: track 58.7 -> 110.0 mm
- net Net-(C102-Pad1): track 14.5 -> 39.6 mm
- net Net-(C101-Pad1): track 27.6 -> 39.3 mm
- net Net-(D110-Pad1): track 0.00 -> 7.62 mm
- net Net-(D112-Pad1): track 0.00 -> 7.62 mm
- net Net-(P101-Pad5): track 0.00 -> 5.08 mm
- net Net-(P101-Pad4): track 0.00 -> 5.08 mm
- net Net-(P101-Pad3): track 0.00 -> 5.08 mm
- net Net-(P101-Pad2): track 0.00 -> 5.08 mm
- net Net-(D109-Pad1): track 0.00 -> 3.81 mm
- net Net-(D111-Pad1): track 0.00 -> 3.81 mm
Other:
- board size 132.1 x 63 mm -> 157.5 x 63 mm

Commit message: 201031
Parts:
- moved P101 261.2 mm to (132.2, 126.0), turned to 0 degrees
- moved R101 258.7 mm to (132.2, 117.1)
- moved R102 253.1 mm to (135.4, 117.1)
- moved R103 246.9 mm to (139.2, 117.1)
- moved R104 241.3 mm to (142.4, 117.1)
- moved C103 233.4 mm to (117.6, 93.0), turned to 270 degrees
- moved D111 223.6 mm to (122.7, 99.3), turned to 270 degrees
- moved D109 221.7 mm to (122.7, 123.4), turned to 90 degrees
- moved D112 215.2 mm to (127.8, 99.3), turned to 270 degrees
- moved D110 213.4 mm to (127.8, 123.4), turned to 90 degrees
- moved R108 200.6 mm to (162.1, 86.6), turned to 90 degrees
- moved R109 198.4 mm to (162.1, 97.4), turned to 90 degrees
- moved R105 195.4 mm to (165.2, 86.6), turned to 90 degrees
- moved U104 194.6 mm to (125.2, 81.5), turned to 90 degrees
- moved U102 193.3 mm to (125.2, 94.9), turned to 90 degrees
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- renumbered U105-JP101 to U106-JP101, U105-JP102 to U106-JP102
Routing:
- net GND: track 110.0 -> 509.0 mm
- net /+5V: track 0.00 -> 127.0 mm
- net Net-(D109-Pad2): track 0.00 -> 118.6 mm
- net Net-(R105-Pad1): track 0.00 -> 96.4 mm
- net Net-(R107-Pad1): track 0.00 -> 78.9 mm
- net Net-(R106-Pad1): track 0.00 -> 71.7 mm
- net Net-(D112-Pad1): track 7.62 -> 52.2 mm
- net Net-(R108-Pad1): track 0.00 -> 44.4 mm, vias 0 -> 1
- net Net-(D111-Pad1): track 3.81 -> 48.2 mm
- net Net-(D109-Pad1): track 3.81 -> 42.1 mm
- net Net-(D110-Pad1): track 7.62 -> 35.5 mm
- net Net-(P107-Pad2): track 0.00 -> 26.1 mm
- net Net-(P105-Pad3): track 0.00 -> 24.7 mm
- net Net-(P105-Pad2): track 0.00 -> 19.6 mm
- net /+3.3V: track 0.00 -> 15.2 mm
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Other:
- board size 157.5 x 63 mm -> 160.5 x 63 mm
- board text added: "DN.: 59/11/3"
- board text added: "MM6D * 2020"
- board text added: "U106"
