File: cad_files/mainboard/mainboard.kicad_pcb (KiCad board)
At the start: 2 copper layers, 160.5 x 63 mm, 62 parts, among them P101 CONN_01X05, P102 CONN_01X02, P103 CONN_01X02, P104 CONN_01X02, P105 CONN_01X03, P106 CONN_01X02, P107 CONN_01X02, P108 CONN_01X02, P109 CONN_01X05, Q101 BC182, Q102 BC182, Q103 BC182, Q104 BC182, Q105 BD137, Q106 BD137, Q107 BD137, Q108 BD137, U101 7805, U102 4N25, U103 4N25, U104 4N25, U105 4N25, U106-JP101 CONN_01X16, U106-JP102 CONN_01X12

Commit message: 201101
Parts:
- moved Q102 2.61 mm to (200.0, 94.1), turned to 0 degrees
- moved Q104 2.56 mm to (213.0, 103.9), turned to 180 degrees
- moved Q103 2.56 mm to (202.4, 103.9), turned to 180 degrees
- moved Q101 2.54 mm to (210.4, 94.1), turned to 0 degrees
Connections:
- Q101 pad 1: Net-(Q101-Pad1) -> Net-(D113-Pad2)
- Q101 pad 3: Net-(D113-Pad2) -> Net-(Q101-Pad3)
- Q102 pad 1: Net-(Q102-Pad1) -> Net-(D114-Pad2)
- Q102 pad 3: Net-(D114-Pad2) -> Net-(Q102-Pad3)
- Q103 pad 1: Net-(Q103-Pad1) -> Net-(D115-Pad2)
- Q103 pad 3: Net-(D115-Pad2) -> Net-(Q103-Pad3)
- Q104 pad 1: Net-(Q104-Pad1) -> Net-(D116-Pad2)
- Q104 pad 3: Net-(D116-Pad2) -> Net-(Q104-Pad3)
- Q105 pad 3: Net-(Q101-Pad1) -> Net-(Q101-Pad3)
- Q106 pad 3: Net-(Q102-Pad1) -> Net-(Q102-Pad3)
- Q107 pad 3: Net-(Q103-Pad1) -> Net-(Q103-Pad3)
- Q108 pad 3: Net-(Q104-Pad1) -> Net-(Q104-Pad3)
Routing:
- net Net-(Q101-Pad3): track 0.00 -> 7.96 mm
- net Net-(Q101-Pad1): track 7.96 -> 0.00 mm
- net Net-(Q102-Pad3): track 0.00 -> 5.50 mm
- net Net-(Q102-Pad1): track 5.50 -> 0.00 mm
- net Net-(Q104-Pad3): track 0.00 -> 5.50 mm
- net Net-(Q104-Pad1): track 5.50 -> 0.00 mm
- net Net-(Q103-Pad3): track 0.00 -> 5.50 mm
- net Net-(Q103-Pad1): track 5.50 -> 0.00 mm

Commit message: 240423
Other:
- board text added: "MM6D * 2023"
- board text removed: "DN.: 59/11/3"
- board text removed: "MM6D * 2020"
Changed lines of the file:
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@@
-(kicad_pcb (version 4) (host pcbnew 4.0.5+dfsg1-4)
+(kicad_pcb (version 20171130) (host pcbnew 5.1.5+dfsg1-2build2)
   (general
-    (links 106)
-    (no_connects 0)
-    (area 68.540143 67.723 241.593858 131.005)
     (thickness 1.6)
-    (drawings 15)
+    (drawings 14)
     (tracks 377)
     (zones 0)
@@
   (page A4)
   (title_block
-    (title "MM6D Remote controlled switching device")
-    (date 2020-06-12)
-    (rev 200612)
-    (company "Pozsar Zsolt - http://www.szerafingomba.hu")
+    (title "MM6D Grow house control device")
+    (date 2024-04-23)
+    (rev 231006)
+    (company "Pozsar Zsolt - http://www.pozsarzs.hu")
     (comment 1 "Main board")
-    (comment 4 "Draw no.: 59/11/3")
   )
   (layers
@@
     (35 F.Paste user)
     (36 B.SilkS user)
-    (37 F.SilkS user hide)
+    (37 F.SilkS user)
     (38 B.Mask user)
     (39 F.Mask user)
@@
     (zone_45_only no)
     (trace_min 0.2)
-    (segment_width 0.2)
-    (edge_width 0.1)
     (via_size 0.6)
     (via_drill 0.4)
@@
     (uvia_min_size 0.2)
     (uvia_min_drill 0.1)
+    (edge_width 0.1)
+    (segment_width 0.2)
     (pcb_text_width 0.3)
     (pcb_text_size 1.5 1.5)
@@
     (visible_elements 7FFEF7FF)
     (pcbplotparams
-      (layerselection 0x00020_00000001)
+      (layerselection 0x010f0_ffffffff)
       (usegerberextensions false)
+      (usegerberattributes false)
+      (usegerberadvancedattributes false)
+      (creategerberjobfile false)
       (excludeedgelayer false)
       (linewidth 0.100000)
-      (plotframeref true)
+      (plotframeref false)
       (viasonmask false)
       (mode 1)
@@
       (hpglpennumber 1)
       (hpglpenspeed 20)
-      (hpglpendiameter 15)
-      (hpglpenoverlay 2)
+      (hpglpendiameter 15.000000)
       (psnegative false)
       (psa4output false)
@@
       (padsonsilk false)
       (subtractmaskfromsilk false)
-      (outputformat 4)
+      (outputformat 1)
       (mirror false)
-      (drillshape 2)
+      (drillshape 0)
       (scaleselection 1)
       (outputdirectory ""))
@@
       (net 2 "Net-(C104-Pad2)"))
     (model Capacitors_ThroughHole.3dshapes/C_Rect_L7_W4.5_P5.wrl
-      (at (xyz 0.098425 0 0))
+      (offset (xyz 2.499994962453842 0 0))
       (scale (xyz 1 1 1))
       (rotate (xyz 0 0 0))
@@
       (net 2 "Net-(C104-Pad2)"))
     (model Socket_Strips.3dshapes/Socket_Strip_Straight_1x02.wrl
-      (at (xyz 0.05 0 0))
+      (offset (xyz 1.269999980926514 0 0))
       (scale (xyz 1 1 1))
       (rotate (xyz 0 0 180))
@@
       (net 4 "Net-(P107-Pad2)"))
     (model Socket_Strips.3dshapes/Socket_Strip_Straight_1x02.wrl
-      (at (xyz 0.05 0 0))
+      (offset (xyz 1.269999980926514 0 0))
       (scale (xyz 1 1 1))
       (rotate (xyz 0 0 180))
@@
       (net 3 GND))
     (model Socket_Strips.3dshapes/Socket_Strip_Straight_1x02.wrl
-      (at (xyz 0.05 0 0))
+      (offset (xyz 1.269999980926514 0 0))
       (scale (xyz 1 1 1))
       (rotate (xyz 0 0 180))
@@
       (net 8 "Net-(P105-Pad3)"))
     (model Socket_Strips.3dshapes/Socket_Strip_Straight_1x03.wrl
-      (at (xyz 0.1 0 0))
+      (offset (xyz 2.539999961853027 0 0))
       (scale (xyz 1 1 1))
       (rotate (xyz 0 0 180))
@@
       (net 57 "Net-(U106-JP101-Pad16)"))
     (model Socket_Strips.3dshapes/Socket_Strip_Straight_1x16.wrl
-      (at (xyz 0.75 0 0))
+      (offset (xyz 19.04999971389771 0 0))
       (scale (xyz 1 1 1))
       (rotate (xyz 0 0 180))
@@
       (net 1 "Net-(C104-Pad1)"))
     (model Socket_Strips.3dshapes/Socket_Strip_Straight_1x12.wrl
-      (at (xyz 0.55 0 0))
+      (offset (xyz 13.96999979019165 0 0))
       (scale (xyz 1 1 1))
       (rotate (xyz 0 0 180))
@@
     (descr "Film Capacitor Length 7mm x Width 4.5mm, Pitch 5mm")
     (tags Capacitor)
-    (fp_text reference C103 (at 7.366 0.254 360) (layer F.SilkS)
+    (fp_text reference C103 (at 7.366 0.254) (layer F.SilkS)
       (effects (font (size 1 1) (thickness 0.15)))
     )
@@
       (net 3 GND))
     (model Capacitors_ThroughHole.3dshapes/C_Rect_L7_W4.5_P5.wrl
-      (at (xyz 0.098425 0 0))
+      (offset (xyz 2.499994962453842 0 0))
       (scale (xyz 1 1 1))
       (rotate (xyz 0 0 0))
@@
       (net 14 "Net-(C101-Pad1)"))
     (model Socket_Strips.3dshapes/Socket_Strip_Straight_1x02.wrl
-      (at (xyz 0.05 0 0))
+      (offset (xyz 1.269999980926514 0 0))
       (scale (xyz 1 1 1))
       (rotate (xyz 0 0 180))
@@
       (net 18 "Net-(D103-Pad2)"))
     (model Socket_Strips.3dshapes/Socket_Strip_Straight_1x02.wrl
-      (at (xyz 0.05 0 0))
+      (offset (xyz 1.269999980926514 0 0))
       (scale (xyz 1 1 1))
       (rotate (xyz 0 0 180))
@@
       (net 20 "Net-(D107-Pad2)"))
     (model Socket_Strips.3dshapes/Socket_Strip_Straight_1x02.wrl
-      (at (xyz 0.05 0 0))
+      (offset (xyz 1.269999980926514 0 0))
       (scale (xyz 1 1 1))
       (rotate (xyz 0 0 180))
@@
       (net 29 "Net-(P101-Pad5)"))
     (model Socket_Strips.3dshapes/Socket_Strip_Straight_1x05.wrl
-      (at (xyz 0.2 0 0))
+      (offset (xyz 5.079999923706055 0 0))
       (scale (xyz 1 1 1))
       (rotate (xyz 0 0 180))
@@
     (descr "Resitance 3 pas")
     (tags R)
-    (fp_text reference R101 (at 0 0 450) (layer F.SilkS)
+    (fp_text reference R101 (at 0 0 90) (layer F.SilkS)
       (effects (font (size 1 1) (thickness 0.15)))
     )
@@
       (net 38 "Net-(D116-Pad2)"))
     (model Socket_Strips.3dshapes/Socket_Strip_Straight_1x05.wrl
-      (at (xyz 0.2 0 0))
+      (offset (xyz 5.079999923706055 0 0))
       (scale (xyz 1 1 1))
       (rotate (xyz 0 0 180))
@@
       (net 34 "Net-(D113-Pad2)"))
     (model TO_SOT_Packages_THT.3dshapes/TO-92_Inline_Narrow_Oval.wrl
-      (at (xyz 0.05 0 0))
+      (offset (xyz 1.269999980926514 0 0))
       (scale (xyz 1 1 1))
       (rotate (xyz 0 0 -90))
@@
       (net 36 "Net-(D114-Pad2)"))
     (model TO_SOT_Packages_THT.3dshapes/TO-92_Inline_Narrow_Oval.wrl
-      (at (xyz 0.05 0 0))
+      (offset (xyz 1.269999980926514 0 0))
       (scale (xyz 1 1 1))
       (rotate (xyz 0 0 -90))
@@
       (net 37 "Net-(D115-Pad2)"))
     (model TO_SOT_Packages_THT.3dshapes/TO-92_Inline_Narrow_Oval.wrl
-      (at (xyz 0.05 0 0))
+      (offset (xyz 1.269999980926514 0 0))
       (scale (xyz 1 1 1))
       (rotate (xyz 0 0 -90))
@@
       (net 38 "Net-(D116-Pad2)"))
     (model TO_SOT_Packages_THT.3dshapes/TO-92_Inline_Narrow_Oval.wrl
-      (at (xyz 0.05 0 0))
+      (offset (xyz 1.269999980926514 0 0))
       (scale (xyz 1 1 1))
       (rotate (xyz 0 0 -90))
@@
     (effects (font (size 1 1) (thickness 0.15)))
   )
-  (gr_text "DN.: 59/11/3" (at 184.404 72.39) (layer F.SilkS)
-    (effects (font (size 1.5 1.5) (thickness 0.3)))
-  )
-  (gr_text "MM6D * 2020" (at 148.082 108.712 90) (layer B.Cu)
+  (gr_text "MM6D * 2023" (at 148.082 108.712 90) (layer B.Cu)
     (effects (font (size 1.5 1.5) (thickness 0.3)) (justify mirror))
   )
