File: cad_files/mainboard/mainboard.sch (KiCad schematic (older format))
At the start: 48 parts, among them P101 CONN_01X05, P102 CONN_01X03, P103 CONN_01X02, P104 CONN_01X02, P105 CONN_01X02, P106 CONN_01X02, P107 CONN_01X05, Q101 BC182, Q102 BC182, Q103 BC182, Q104 BC182, Q105 BD137, Q106 BD137, Q107 BD137, Q108 BD137, U101 4N25, U102 4N25, U103 4N25, U104 4N25, U105-JP101 CONN_01X16, U105-JP102 CONN_01X12, U106 7805

Commit message: 201029
Parts:
- removed D105: 1N4001, Diodes_THT:Diode_DO-41_SOD81_Horizontal_RM10, symbol D
- added C102: 470u, Capacitors_THT:C_Radial_D8_L11.5_P3.5, symbol device:CP_Small
- added D101, D102, D103, D104, D105, D106, D107, D108: 1N4001, Diodes_THT:Diode_DO-41_SOD81_Horizontal_RM10, symbol diode
- added P101, P103: CONN_01X02, Socket_Strips:Socket_Strip_Straight_1x02, symbol CONN_01X02
- C103: footprint (none) -> Capacitors_THT:C_Rect_L7_W4.5_P5
- U101: renamed from U106; footprint (none) -> TO_SOT_Packages_THT:TO-220_Neutral123_Horizontal_LargePads
- renumbered C102 to C104, D101 to D109, D102 to D110, D103 to D111, D104 to D112, D106 to D113, D107 to D114, D108 to D115, D109 to D116, P103 to P102, P101 to P104, P107 to P105, P102 to P106, P104 to P107, P105 to P108, P106 to P109, U101 to U102, U102 to U103, U103 to U104, U104 to U105
Connections:
- wire segments 158 -> 186
Other:
- note added: "U106"
- note removed: "12V DC"
- note removed: "Accu"
- note removed: "Active\n LED"
- note removed: "Console"
- note removed: "Inputs"
- note removed: "Outputs"
- note removed: "Piezo\nspeaker"
- note removed: "U105"
- moved on the sheet: C103, C104, P102, P104, P105, P106, P107, P108, P109, Q101, Q102, Q103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

Commit message: 201030
Parts:
- removed D101, D102, D103, D104, D105, D106, D107, D108, D109, D110, D111, D112: 1N4001, Diodes_THT:Diode_DO-41_SOD81_Horizontal_RM10, symbol diode
- removed D113, D114, D115, D116: 1N4007, Diodes_THT:Diode_DO-41_SOD81_Horizontal_RM10, symbol diode
- added D101, D102, D103, D104, D105, D106, D107, D108, D109, D110, D111, D112: 1N4001, Diodes_THT:Diode_DO-41_SOD81_Horizontal_RM10, symbol D
- added D113, D114, D115, D116: 1N4007, Diodes_THT:Diode_DO-41_SOD81_Horizontal_RM10, symbol D
- renumbered P104 to P101, P103 to P102, P101 to P103, P102 to P104, P106 to P105, P107 to P106, P108 to P107, P109 to P108, P105 to P109

Commit message: 201031
Parts:
- renumbered U105-JP101 to U106-JP101, U105-JP102 to U106-JP102
Changed lines of the file:
@@
 	6075 2475 5625 2475
 $Comp
-L CONN_01X16 U105-JP101
+L CONN_01X16 U106-JP101
 U 1 1 5F19AC96
 P 5525 3275
-F 0 "U105-JP101" H 5525 2375 50  0000 C CNN
+F 0 "U106-JP101" H 5525 2375 50  0000 C CNN
 F 1 "CONN_01X16" V 5625 3275 50  0001 C CNN
 F 2 "Socket_Strips:Socket_Strip_Straight_1x16" H 5525 3275 50  0001 C CNN
@@
 $EndComp
 $Comp
-L CONN_01X12 U105-JP102
+L CONN_01X12 U106-JP102
 U 1 1 5F19AC49
 P 6175 3475
-F 0 "U105-JP102" H 6175 4575 50  0000 C CNN
+F 0 "U106-JP102" H 6175 4575 50  0000 C CNN
 F 1 "CONN_01X12" V 6275 3475 50  0001 C CNN
 F 2 "Socket_Strips:Socket_Strip_Straight_1x12" H 6175 3475 50  0001 C CNN

Commit message: 201101
Parts:
- removed Q101, Q102, Q103, Q104: BC182, TO_SOT_Packages_THT:TO-92_Inline_Narrow_Oval, symbol Q_NPN_EBC
- added Q101, Q102, Q103, Q104: BC182, TO_SOT_Packages_THT:TO-92_Molded_Narrow, symbol Q_NPN_CBE
Connections:
- net at R111.2: now also Q101.2 (B)
- net at D115.2 (A), P109.4 (P4), Q107.2 (C): now also Q103.1 (C)
- net at Q107.3 (B): now also Q103.3 (E)
- net at D116.2 (A), P109.5 (P5), Q108.2 (C): now also Q104.1 (C)
- net at Q108.3 (B): now also Q104.3 (E)
- net at D114.2 (A), P109.3 (P3), Q106.2 (C): now also Q102.1 (C)
- net at Q106.3 (B): now also Q102.3 (E)
- net at D113.2 (A), P109.2 (P2), Q105.2 (C): now also Q101.1 (C)
- net at Q105.3 (B): now also Q101.3 (E)
- net at R112.2: now also Q102.2 (B)
- net at R113.2: now also Q103.2 (B)
- net at R114.2: now also Q104.2 (B)
Changed lines of the file:
@@
 	4625 1475 4625 1625
 Wire Wire Line
-	4175 1475 5125 1475
+	5125 1475 4175 1475
 Wire Wire Line
 	4175 1475 4175 1625
@@
 	5125 2825 5125 5275
 $Comp
-L pzs_others:0V #PWR06
+L pzs_others:0V #PWR04
 U 1 1 5F1E7647
 P 4625 5275
-F 0 "#PWR06" H 4625 5025 50  0001 C CNN
+F 0 "#PWR04" H 4625 5025 50  0001 C CNN
 F 1 "0V" H 4625 5125 50  0001 C CNN
 F 2 "" H 4625 5275 50  0000 C CNN
@@
 $EndComp
 $Comp
-L pzs_others:0V #PWR04
+L pzs_others:0V #PWR05
 U 1 1 5F19FE91
 P 4825 1275
-F 0 "#PWR04" H 4825 1025 50  0001 C CNN
+F 0 "#PWR05" H 4825 1025 50  0001 C CNN
 F 1 "0V" H 4825 1125 50  0001 C CNN
 F 2 "" H 4825 1275 50  0000 C CNN
@@
 NoConn ~ 3800 2125
 $Comp
-L pzs_others:0V #PWR03
+L pzs_others:0V #PWR06
 U 1 1 5F1AA249
 P 4175 5275
-F 0 "#PWR03" H 4175 5025 50  0001 C CNN
+F 0 "#PWR06" H 4175 5025 50  0001 C CNN
 F 1 "0V" H 4175 5125 50  0001 C CNN
 F 2 "" H 4175 5275 50  0000 C CNN
@@
 NoConn ~ 5325 2525
 $Comp
-L pzs_others:0V #PWR01
+L pzs_others:0V #PWR07
 U 1 1 5EEE442D
 P 5125 5275
-F 0 "#PWR01" H 5125 5025 50  0001 C CNN
+F 0 "#PWR07" H 5125 5025 50  0001 C CNN
 F 1 "0V" H 5125 5125 50  0001 C CNN
 F 2 "" H 5125 5275 50  0000 C CNN
@@
 	1625 5525 2675 5525
 $Comp
-L pzs_others:0V #PWR010
+L pzs_others:0V #PWR08
 U 1 1 5F9BD0C0
 P 2675 5525
-F 0 "#PWR010" H 2675 5275 50  0001 C CNN
+F 0 "#PWR08" H 2675 5275 50  0001 C CNN
 F 1 "0V" H 2675 5375 50  0001 C CNN
 F 2 "" H 2675 5525 50  0000 C CNN
@@
 $EndComp
 $Comp
-L pzs_others:0V #PWR08
+L pzs_others:0V #PWR010
 U 1 1 5F7F7EA1
 P 2675 6375
-F 0 "#PWR08" H 2675 6125 50  0001 C CNN
+F 0 "#PWR010" H 2675 6125 50  0001 C CNN
 F 1 "0V" H 2675 6225 50  0001 C CNN
 F 2 "" H 2675 6375 50  0000 C CNN
@@
 	8650 5075 8650 5275
 $Comp
-L Q_NPN_EBC Q104
-U 1 1 5F1A19FD
-P 8150 4575
-F 0 "Q104" H 8350 4625 50  0000 L CNN
-F 1 "BC182" H 8350 4525 50  0000 L CNN
-F 2 "TO_SOT_Packages_THT:TO-92_Inline_Narrow_Oval" H 8350 4675 50  0001 C CNN
-F 3 "" H 8150 4575 50  0000 C CNN
-	1    8150 4575
-	1    0    0    -1
-$EndComp
-$Comp
-L Q_NPN_EBC Q103
-U 1 1 5F1A1931
-P 8150 3625
-F 0 "Q103" H 8350 3675 50  0000 L CNN
-F 1 "BC182" H 8350 3575 50  0000 L CNN
-F 2 "TO_SOT_Packages_THT:TO-92_Inline_Narrow_Oval" H 8350 3725 50  0001 C CNN
-F 3 "" H 8150 3625 50  0000 C CNN
-	1    8150 3625
-	1    0    0    -1
-$EndComp
-$Comp
-L Q_NPN_EBC Q102
-U 1 1 5F1A185C
-P 8150 2675
-F 0 "Q102" H 8350 2725 50  0000 L CNN
-F 1 "BC182" H 8350 2625 50  0000 L CNN
-F 2 "TO_SOT_Packages_THT:TO-92_Inline_Narrow_Oval" H 8350 2775 50  0001 C CNN
-F 3 "" H 8150 2675 50  0000 C CNN
-	1    8150 2675
-	1    0    0    -1
-$EndComp
-$Comp
-L Q_NPN_EBC Q101
-U 1 1 5F1A151F
-P 8150 1725
-F 0 "Q101" H 8350 1775 50  0000 L CNN
-F 1 "BC182" H 8350 1675 50  0000 L CNN
-F 2 "TO_SOT_Packages_THT:TO-92_Inline_Narrow_Oval" H 8350 1825 50  0001 C CNN
-F 3 "" H 8150 1725 50  0000 C CNN
-	1    8150 1725
-	1    0    0    -1
-$EndComp
-$Comp
 L Q_NPN_ECB Q105
 U 1 1 5F1A10F1
@@
 $EndComp
 $Comp
-L pzs_others:0V #PWR02
+L pzs_others:0V #PWR011
 U 1 1 5EF79B48
 P 8650 5275
-F 0 "#PWR02" H 8650 5025 50  0001 C CNN
+F 0 "#PWR011" H 8650 5025 50  0001 C CNN
 F 1 "0V" H 8650 5125 50  0001 C CNN
 F 2 "" H 8650 5275 50  0000 C CNN
@@
 	1    0    0    -1
 $EndComp
+$Comp
+L Q_NPN_CBE Q101
+U 1 1 5F9EAEA4
+P 8150 1725
+F 0 "Q101" H 8350 1775 50  0000 L CNN
+F 1 "BC182" H 8350 1675 50  0000 L CNN
+F 2 "TO_SOT_Packages_THT:TO-92_Molded_Narrow" H 8350 1825 50  0001 C CNN
+F 3 "" H 8150 1725 50  0000 C CNN
+	1    8150 1725
+	1    0    0    -1
+$EndComp
+$Comp
+L Q_NPN_CBE Q102
+U 1 1 5F9EB64D
+P 8150 2675
+F 0 "Q102" H 8350 2725 50  0000 L CNN
+F 1 "BC182" H 8350 2625 50  0000 L CNN
+F 2 "TO_SOT_Packages_THT:TO-92_Molded_Narrow" H 8350 2775 50  0001 C CNN
+F 3 "" H 8150 2675 50  0000 C CNN
+	1    8150 2675
+	1    0    0    -1
+$EndComp
+$Comp
+L Q_NPN_CBE Q103
+U 1 1 5F9EB737
+P 8150 3625
+F 0 "Q103" H 8350 3675 50  0000 L CNN
+F 1 "BC182" H 8350 3575 50  0000 L CNN
+F 2 "TO_SOT_Packages_THT:TO-92_Molded_Narrow" H 8350 3725 50  0001 C CNN
+F 3 "" H 8150 3625 50  0000 C CNN
+	1    8150 3625
+	1    0    0    -1
+$EndComp
+$Comp
+L Q_NPN_CBE Q104
+U 1 1 5F9EB816
+P 8150 4575
+F 0 "Q104" H 8350 4625 50  0000 L CNN
+F 1 "BC182" H 8350 4525 50  0000 L CNN
+F 2 "TO_SOT_Packages_THT:TO-92_Molded_Narrow" H 8350 4675 50  0001 C CNN
+F 3 "" H 8150 4575 50  0000 C CNN
+	1    8150 4575
+	1    0    0    -1
+$EndComp

Commit message: 201226
Parts:
- C102: value 470u -> 1000u
- C103: value 4.7u -> 1u
- R101, R102, R103, R104: value 1.5k -> 9.1k
- R110: value 390 -> 750
- R111, R112, R113, R114: value 1k -> 1.5k
Connections:
- no-connect marks 16 -> 17
Changed lines of the file:
@@
 U 1 1 5F1AEBA9
 P 7500 2150
-F 0 "R110" H 7675 2200 50  0000 C CNN
-F 1 "390" H 7650 2125 50  0000 C CNN
+F 0 "R110" H 7700 2075 50  0000 C CNN
+F 1 "750" H 7675 2225 50  0000 C CNN
 F 2 "Discret:R3" V 7430 2150 50  0001 C CNN
 F 3 "" H 7500 2150 50  0000 C CNN
@@
 Connection ~ 4175 4725
 Wire Wire Line
-	5125 2625 5125 1475
-Wire Wire Line
-	5325 2625 5125 2625
+	5125 1475 5125 2625
+Wire Wire Line
+	5125 2625 5325 2625
 Wire Wire Line
 	5125 2825 5325 2825
@@
 	4625 1475 4625 1625
 Wire Wire Line
-	5125 1475 4175 1475
+	4175 1475 5125 1475
 Wire Wire Line
 	4175 1475 4175 1625
@@
 Connection ~ 4175 3925
 Wire Wire Line
-	3800 3925 4175 3925
+	4175 3925 3800 3925
 Wire Wire Line
 	4175 4725 3800 4725
@@
 P 2575 6875
 F 0 "C102" H 2625 7000 50  0000 L CNN
-F 1 "470u" H 2625 6775 50  0000 L CNN
+F 1 "1000u" H 2625 6775 50  0000 L CNN
 F 2 "Capacitors_THT:C_Radial_D8_L11.5_P3.5" H 2575 6875 50  0001 C CNN
 F 3 "" H 2575 6875 50  0000 C CNN
@@
 P 3575 6875
 F 0 "C103" H 3650 7025 50  0000 L CNN
-F 1 "4.7u" H 3650 6775 50  0000 L CNN
+F 1 "1u" H 3650 6775 50  0000 L CNN
 F 2 "Capacitors_THT:C_Rect_L7_W4.5_P5" H 3575 6875 50  0001 C CNN
 F 3 "" H 3575 6875 50  0001 C CNN
@@
 U 1 1 5F9C8E0D
 P 2850 4775
-F 0 "D112" V 2900 4925 50  0000 C CNN
+F 0 "D112" V 2900 4950 50  0000 C CNN
 F 1 "1N4001" V 3225 4775 50  0000 C CNN
 F 2 "Diodes_THT:Diode_DO-41_SOD81_Horizontal_RM10" H 2850 4775 50  0001 C CNN
@@
 U 1 1 5F9C8CC6
 P 2850 3950
-F 0 "D111" V 2900 4100 50  0000 C CNN
+F 0 "D111" V 2900 4125 50  0000 C CNN
 F 1 "1N4001" V 3225 3950 50  0000 C CNN
 F 2 "Diodes_THT:Diode_DO-41_SOD81_Horizontal_RM10" H 2850 3950 50  0001 C CNN
@@
 U 1 1 5F9C8BD4
 P 2850 3150
-F 0 "D110" V 2900 3300 50  0000 C CNN
+F 0 "D110" V 2900 3325 50  0000 C CNN
 F 1 "1N4001" V 3225 3150 50  0000 C CNN
 F 2 "Diodes_THT:Diode_DO-41_SOD81_Horizontal_RM10" H 2850 3150 50  0001 C CNN
@@
 U 1 1 5F9C7564
 P 2850 2375
-F 0 "D109" V 2900 2525 50  0000 C CNN
+F 0 "D109" V 2900 2550 50  0000 C CNN
 F 1 "1N4001" V 3225 2375 50  0000 C CNN
 F 2 "Diodes_THT:Diode_DO-41_SOD81_Horizontal_RM10" H 2850 2375 50  0001 C CNN
@@
 P 2550 4525
 F 0 "R104" V 2450 4525 50  0000 C CNN
-F 1 "1.5k" V 2650 4525 50  0000 C CNN
+F 1 "9.1k" V 2650 4525 50  0000 C CNN
 F 2 "Discret:R3" V 2480 4525 50  0001 C CNN
 F 3 "" H 2550 4525 50  0000 C CNN
@@
 P 2550 3725
 F 0 "R103" V 2450 3725 50  0000 C CNN
-F 1 "1.5k" V 2650 3725 50  0000 C CNN
+F 1 "9.1k" V 2650 3725 50  0000 C CNN
 F 2 "Discret:R3" V 2480 3725 50  0001 C CNN
 F 3 "" H 2550 3725 50  0000 C CNN
@@
 P 2550 2925
 F 0 "R102" V 2450 2925 50  0000 C CNN
-F 1 "1.5k" V 2650 2925 50  0000 C CNN
+F 1 "9.1k" V 2650 2925 50  0000 C CNN
 F 2 "Discret:R3" V 2480 2925 50  0001 C CNN
 F 3 "" H 2550 2925 50  0000 C CNN
@@
 P 2550 2125
 F 0 "R101" V 2450 2125 50  0000 C CNN
-F 1 "1.5k" V 2650 2125 50  0000 C CNN
+F 1 "9.1k" V 2650 2125 50  0000 C CNN
 F 2 "Discret:R3" V 2480 2125 50  0001 C CNN
 F 3 "" H 2550 2125 50  0000 C CNN
@@
 P 7750 4575
 F 0 "R114" V 7650 4575 50  0000 C CNN
-F 1 "1k" V 7850 4575 50  0000 C CNN
+F 1 "1.5k" V 7850 4575 50  0000 C CNN
 F 2 "Discret:R3" V 7680 4575 50  0001 C CNN
 F 3 "" H 7750 4575 50  0000 C CNN
@@
 P 7750 3625
 F 0 "R113" V 7650 3625 50  0000 C CNN
-F 1 "1k" V 7850 3625 50  0000 C CNN
+F 1 "1.5k" V 7850 3625 50  0000 C CNN
 F 2 "Discret:R3" V 7680 3625 50  0001 C CNN
 F 3 "" H 7750 3625 50  0000 C CNN
@@
 P 7750 2675
 F 0 "R112" V 7650 2675 50  0000 C CNN
-F 1 "1k" V 7850 2675 50  0000 C CNN
+F 1 "1.5k" V 7850 2675 50  0000 C CNN
 F 2 "Discret:R3" V 7680 2675 50  0001 C CNN
 F 3 "" H 7750 2675 50  0000 C CNN
@@
 P 7750 1725
 F 0 "R111" V 7650 1725 50  0000 C CNN
-F 1 "1k" V 7850 1725 50  0000 C CNN
+F 1 "1.5k" V 7850 1725 50  0000 C CNN
 F 2 "Discret:R3" V 7680 1725 50  0001 C CNN
 F 3 "" H 7750 1725 50  0000 C CNN
@@
 	1    0    0    -1
 $EndComp
+NoConn ~ 2725 6975
 $EndSCHEMATC

Commit message: 240423
Parts:
- C101, C102, C103, C104: symbol device:CP_Small -> mainboard-rescue:device_CP_Small
- D101, D102, D103, D104, D105, D106, D107, D108, D109, D110, D111, D112, D113, D114, D115, D116: symbol D -> mainboard-rescue:D
- P101, P109: symbol CONN_01X05 -> mainboard-rescue:CONN_01X05
- P102, P103, P104, P106, P107, P108: symbol CONN_01X02 -> mainboard-rescue:CONN_01X02
- P105: symbol CONN_01X03 -> mainboard-rescue:CONN_01X03
- Q101, Q102, Q103, Q104: symbol Q_NPN_CBE -> mainboard-rescue:Q_NPN_CBE
- Q105, Q106, Q107, Q108: symbol Q_NPN_ECB -> mainboard-rescue:Q_NPN_ECB
- R101, R102, R103, R104, R105, R106, R107, R108, R109, R110, R111, R112, R113, R114: symbol R -> mainboard-rescue:R
- U101: symbol 7805 -> mainboard-rescue:7805
- U102, U103, U104, U105: symbol 4N25 -> mainboard-rescue:4N25
- U106-JP101: symbol CONN_01X16 -> mainboard-rescue:CONN_01X16
- U106-JP102: symbol CONN_01X12 -> mainboard-rescue:CONN_01X12
