File: cad_files/display/display.kicad_pcb (KiCad board)
At the start: 2 copper layers, 80 x 71.1 mm, 33 parts, among them P201 CONN_01X02, P202 CONN_01X01, P203 CONN_01X01, P204 CONN_01X06, P205 CONN_01X03, P206 CONN_01X03, P207 CONN_01X03, P208 CONN_01X01, P209 CONN_01X01

Commit message: 201029
Parts:
- moved P205 4.83 mm to (110.2, 68.3), turned to 90 degrees
- moved P201 2.29 mm to (110.2, 124.2), turned to 90 degrees
Connections:
- P201 pad 1: Net-(D209-Pad2) -> Net-(D209-Pad1)
- P201 pad 2: Net-(D209-Pad1) -> Net-(D209-Pad2)
- P205 pad 1: Net-(D212-Pad2) -> Net-(D201-Pad1)
- P205 pad 3: Net-(D201-Pad1) -> Net-(D212-Pad2)
Changed lines of the file:
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@@
     (visible_elements 7FFFFFFF)
     (pcbplotparams
-      (layerselection 0x01060_80000000)
+      (layerselection 0x00020_00000000)
       (usegerberextensions false)
       (excludeedgelayer false)
       (linewidth 0.100000)
-      (plotframeref false)
+      (plotframeref true)
       (viasonmask false)
       (mode 1)
@@
       (padsonsilk false)
       (subtractmaskfromsilk false)
-      (outputformat 1)
+      (outputformat 4)
       (mirror false)
-      (drillshape 0)
+      (drillshape 2)
       (scaleselection 1)
       (outputdirectory ""))
@@
   )
   (module Socket_Strips:Socket_Strip_Straight_1x02 (layer F.Cu)
-    (at 110.236 121.92 270)
+    (at 110.236 124.206 90)
     (descr "Through hole socket strip")
     (tags "socket strip")
-    (fp_text reference P201 (at 1.27 -2.54 270) (layer F.SilkS)
-      (effects (font (size 1 1) (thickness 0.15)))
-    )
-    (fp_text value CONN_01X02 (at 1.27 2.54 270) (layer F.Fab) hide
+    (fp_text reference P201 (at 1.27 -2.54 90) (layer F.SilkS)
+      (effects (font (size 1 1) (thickness 0.15)))
+    )
+    (fp_text value CONN_01X02 (at 1.27 2.54 90) (layer F.Fab) hide
       (effects (font (size 1 1) (thickness 0.15)))
     )
@@
     (fp_line (start 1.27 -1.27) (end 3.81 -1.27) (layer F.SilkS) (width 0.15))
     (fp_line (start 3.81 -1.27) (end 3.81 1.27) (layer F.SilkS) (width 0.15))
-    (pad 1 thru_hole rect (at 0 0 270) (size 2.032 2.032) (drill 1.00076) (layers *.Cu *.Mask)
+    (pad 1 thru_hole rect (at 0 0 90) (size 2.032 2.032) (drill 1.00076) (layers *.Cu *.Mask)
+      (net 16 "Net-(D209-Pad1)"))
+    (pad 2 thru_hole oval (at 2.54 0 90) (size 2.032 2.032) (drill 1.00076) (layers *.Cu *.Mask)
       (net 17 "Net-(D209-Pad2)"))
-    (pad 2 thru_hole oval (at 2.54 0 270) (size 2.032 2.032) (drill 1.00076) (layers *.Cu *.Mask)
-      (net 16 "Net-(D209-Pad1)"))
     (model Socket_Strips.3dshapes/Socket_Strip_Straight_1x02.wrl
       (at (xyz 0.05 0 0))
@@
   )
   (module Socket_Strips:Socket_Strip_Straight_1x03 (layer F.Cu)
-    (at 110.236 63.5 270)
+    (at 110.236 68.326 90)
     (descr "Through hole socket strip")
     (tags "socket strip")
-    (fp_text reference P205 (at 2.794 -2.54 270) (layer F.SilkS)
-      (effects (font (size 1 1) (thickness 0.15)))
-    )
-    (fp_text value CONN_01X03 (at 2.54 2.54 270) (layer F.Fab) hide
+    (fp_text reference P205 (at 2.794 -2.54 90) (layer F.SilkS)
+      (effects (font (size 1 1) (thickness 0.15)))
+    )
+    (fp_text value CONN_01X03 (at 2.54 2.54 90) (layer F.Fab) hide
       (effects (font (size 1 1) (thickness 0.15)))
     )
@@
     (fp_line (start 6.35 1.27) (end 1.27 1.27) (layer F.SilkS) (width 0.15))
     (fp_line (start 1.27 1.27) (end 1.27 -1.27) (layer F.SilkS) (width 0.15))
-    (pad 1 thru_hole rect (at 0 0 270) (size 1.7272 2.032) (drill 1.00076) (layers *.Cu *.Mask)
+    (pad 1 thru_hole rect (at 0 0 90) (size 1.7272 2.032) (drill 1.00076) (layers *.Cu *.Mask)
+      (net 3 "Net-(D201-Pad1)"))
+    (pad 2 thru_hole oval (at 2.54 0 90) (size 1.7272 2.032) (drill 1.00076) (layers *.Cu *.Mask)
+      (net 24 "Net-(P205-Pad2)"))
+    (pad 3 thru_hole oval (at 5.08 0 90) (size 1.7272 2.032) (drill 1.00076) (layers *.Cu *.Mask)
       (net 20 "Net-(D212-Pad2)"))
-    (pad 2 thru_hole oval (at 2.54 0 270) (size 1.7272 2.032) (drill 1.00076) (layers *.Cu *.Mask)
-      (net 24 "Net-(P205-Pad2)"))
-    (pad 3 thru_hole oval (at 5.08 0 270) (size 1.7272 2.032) (drill 1.00076) (layers *.Cu *.Mask)
-      (net 3 "Net-(D201-Pad1)"))
     (model Socket_Strips.3dshapes/Socket_Strip_Straight_1x03.wrl
       (at (xyz 0.1 0 0))

Commit message: 240423
Other:
- board text added: "MM6D 2023"
- board text removed: "DN: 59/11/5"
- board text removed: "MM6D 2020"
Changed lines of the file:
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@@
-(kicad_pcb (version 4) (host pcbnew 4.0.5+dfsg1-4)
+(kicad_pcb (version 20171130) (host pcbnew 5.1.5+dfsg1-2build2)
   (general
-    (links 39)
-    (no_connects 6)
-    (area 104.689 58.090999 185.241001 129.361001)
     (thickness 1.6)
-    (drawings 12)
+    (drawings 11)
     (tracks 66)
     (zones 0)
@@
   (page A4)
   (title_block
-    (title "MM6D Remote controlled switching device")
-    (date 2020-10-26)
-    (rev 200612)
-    (company "Pozsar Zsolt - http://www.szerafingomba.hu")
+    (title "MM6D Grow house control device")
+    (date 2024-04-23)
+    (rev 231006)
+    (company "Pozsar Zsolt - http://www.pozsarzs.hu")
     (comment 1 "Display board")
-    (comment 4 "Draw no.: 59/11/5")
   )
   (layers
@@
     (zone_45_only no)
     (trace_min 0.2)
-    (segment_width 0.2)
-    (edge_width 0.15)
     (via_size 0.6)
     (via_drill 0.4)
@@
     (uvia_min_size 0.2)
     (uvia_min_drill 0.1)
+    (edge_width 0.15)
+    (segment_width 0.2)
     (pcb_text_width 0.3)
     (pcb_text_size 1.5 1.5)
@@
     (visible_elements 7FFFFFFF)
     (pcbplotparams
-      (layerselection 0x00020_00000000)
+      (layerselection 0x010e0_ffffffff)
       (usegerberextensions false)
+      (usegerberattributes false)
+      (usegerberadvancedattributes false)
+      (creategerberjobfile false)
       (excludeedgelayer false)
       (linewidth 0.100000)
-      (plotframeref true)
+      (plotframeref false)
       (viasonmask false)
       (mode 1)
@@
       (hpglpennumber 1)
       (hpglpenspeed 20)
-      (hpglpendiameter 15)
-      (hpglpenoverlay 2)
+      (hpglpendiameter 15.000000)
       (psnegative false)
       (psa4output false)
@@
       (padsonsilk false)
       (subtractmaskfromsilk false)
-      (outputformat 4)
+      (outputformat 1)
       (mirror false)
-      (drillshape 2)
+      (drillshape 0)
       (scaleselection 1)
       (outputdirectory ""))
@@
       (net 2 "Net-(BT201-Pad2)"))
     (model Socket_Strips.3dshapes/Socket_Strip_Straight_1x02.wrl
-      (at (xyz 0.05 0 0))
+      (offset (xyz 1.269999980926514 0 0))
       (scale (xyz 1 1 1))
       (rotate (xyz 0 0 180))
@@
       (net 4 "Net-(D201-Pad2)"))
     (model LEDs.3dshapes/LED-5MM.wrl
-      (at (xyz 0.05 0 0))
+      (offset (xyz 1.269999980926514 0 0))
       (scale (xyz 1 1 1))
       (rotate (xyz 0 0 90))
@@
       (net 6 "Net-(D202-Pad2)"))
     (model LEDs.3dshapes/LED-5MM.wrl
-      (at (xyz 0.05 0 0))
+      (offset (xyz 1.269999980926514 0 0))
       (scale (xyz 1 1 1))
       (rotate (xyz 0 0 90))
@@
       (net 7 "Net-(D203-Pad2)"))
     (model LEDs.3dshapes/LED-5MM.wrl
-      (at (xyz 0.05 0 0))
+      (offset (xyz 1.269999980926514 0 0))
       (scale (xyz 1 1 1))
       (rotate (xyz 0 0 90))
@@
       (net 9 "Net-(D204-Pad2)"))
     (model LEDs.3dshapes/LED-5MM.wrl
-      (at (xyz 0.05 0 0))
+      (offset (xyz 1.269999980926514 0 0))
       (scale (xyz 1 1 1))
       (rotate (xyz 0 0 90))
@@
       (net 11 "Net-(D205-Pad2)"))
     (model LEDs.3dshapes/LED-5MM.wrl
-      (at (xyz 0.05 0 0))
+      (offset (xyz 1.269999980926514 0 0))
       (scale (xyz 1 1 1))
       (rotate (xyz 0 0 90))
@@
       (net 13 "Net-(D206-Pad2)"))
     (model LEDs.3dshapes/LED-5MM.wrl
-      (at (xyz 0.05 0 0))
+      (offset (xyz 1.269999980926514 0 0))
       (scale (xyz 1 1 1))
       (rotate (xyz 0 0 90))
@@
       (net 14 "Net-(D207-Pad2)"))
     (model LEDs.3dshapes/LED-5MM.wrl
-      (at (xyz 0.05 0 0))
+      (offset (xyz 1.269999980926514 0 0))
       (scale (xyz 1 1 1))
       (rotate (xyz 0 0 90))
@@
       (net 15 "Net-(D208-Pad2)"))
     (model LEDs.3dshapes/LED-5MM.wrl
-      (at (xyz 0.05 0 0))
+      (offset (xyz 1.269999980926514 0 0))
       (scale (xyz 1 1 1))
       (rotate (xyz 0 0 90))
@@
       (net 17 "Net-(D209-Pad2)"))
     (model LEDs.3dshapes/LED-5MM.wrl
-      (at (xyz 0.05 0 0))
+      (offset (xyz 1.269999980926514 0 0))
       (scale (xyz 1 1 1))
       (rotate (xyz 0 0 90))
@@
       (net 17 "Net-(D209-Pad2)"))
     (model Socket_Strips.3dshapes/Socket_Strip_Straight_1x02.wrl
-      (at (xyz 0.05 0 0))
+      (offset (xyz 1.269999980926514 0 0))
       (scale (xyz 1 1 1))
       (rotate (xyz 0 0 180))
@@
     (descr "Through hole socket strip")
     (tags "socket strip")
-    (fp_text reference P203 (at -2.54 0 360) (layer F.SilkS)
-      (effects (font (size 1 1) (thickness 0.15)))
-    )
-    (fp_text value CONN_01X01 (at 2.54 0 360) (layer F.Fab) hide
+    (fp_text reference P203 (at -2.54 0) (layer F.SilkS)
+      (effects (font (size 1 1) (thickness 0.15)))
+    )
+    (fp_text value CONN_01X01 (at 2.54 0) (layer F.Fab) hide
       (effects (font (size 1 1) (thickness 0.15)))
     )
@@
       (net 12 "Net-(D206-Pad1)"))
     (model Socket_Strips.3dshapes/Socket_Strip_Straight_1x06.wrl
-      (at (xyz 0.25 0 0))
+      (offset (xyz 6.349999904632568 0 0))
       (scale (xyz 1 1 1))
       (rotate (xyz 0 0 180))
@@
       (net 18 /+12V))
     (model Socket_Strips.3dshapes/Socket_Strip_Straight_1x03.wrl
-      (at (xyz 0.1 0 0))
+      (offset (xyz 2.539999961853027 0 0))
       (scale (xyz 1 1 1))
       (rotate (xyz 0 0 180))
@@
       (net 2 "Net-(BT201-Pad2)"))
     (model Socket_Strips.3dshapes/Socket_Strip_Straight_1x03.wrl
-      (at (xyz 0.1 0 0))
+      (offset (xyz 2.539999961853027 0 0))
       (scale (xyz 1 1 1))
       (rotate (xyz 0 0 180))
@@
       (net 21 "Net-(D212-Pad1)"))
     (model Resistors_ThroughHole.3dshapes/Resistor_Horizontal_RM15mm.wrl
-      (at (xyz 0.295 0 0))
+      (offset (xyz 7.49299988746643 0 0))
       (scale (xyz 0.395 0.4 0.4))
       (rotate (xyz 0 0 0))
@@
       (net 18 /+12V))
     (model Resistors_ThroughHole.3dshapes/Resistor_Horizontal_RM15mm.wrl
-      (at (xyz 0.295 0 0))
+      (offset (xyz 7.49299988746643 0 0))
       (scale (xyz 0.395 0.4 0.4))
       (rotate (xyz 0 0 0))
@@
       (net 18 /+12V))
     (model Resistors_ThroughHole.3dshapes/Resistor_Horizontal_RM15mm.wrl
-      (at (xyz 0.295 0 0))
+      (offset (xyz 7.49299988746643 0 0))
       (scale (xyz 0.395 0.4 0.4))
       (rotate (xyz 0 0 0))
@@
       (net 18 /+12V))
     (model Resistors_ThroughHole.3dshapes/Resistor_Horizontal_RM15mm.wrl
-      (at (xyz 0.295 0 0))
+      (offset (xyz 7.49299988746643 0 0))
       (scale (xyz 0.395 0.4 0.4))
       (rotate (xyz 0 0 0))
@@
       (net 18 /+12V))
     (model Resistors_ThroughHole.3dshapes/Resistor_Horizontal_RM15mm.wrl
-      (at (xyz 0.295 0 0))
+      (offset (xyz 7.49299988746643 0 0))
       (scale (xyz 0.395 0.4 0.4))
       (rotate (xyz 0 0 0))
@@
       (net 18 /+12V))
     (model Resistors_ThroughHole.3dshapes/Resistor_Horizontal_RM15mm.wrl
-      (at (xyz 0.295 0 0))
+      (offset (xyz 7.49299988746643 0 0))
       (scale (xyz 0.395 0.4 0.4))
       (rotate (xyz 0 0 0))
@@
       (net 14 "Net-(D207-Pad2)"))
     (model Resistors_ThroughHole.3dshapes/Resistor_Horizontal_RM15mm.wrl
-      (at (xyz 0.295 0 0))
+      (offset (xyz 7.49299988746643 0 0))
       (scale (xyz 0.395 0.4 0.4))
       (rotate (xyz 0 0 0))
@@
       (net 23 "Net-(P209-Pad1)"))
     (model Resistors_ThroughHole.3dshapes/Resistor_Horizontal_RM15mm.wrl
-      (at (xyz 0.295 0 0))
+      (offset (xyz 7.49299988746643 0 0))
       (scale (xyz 0.395 0.4 0.4))
       (rotate (xyz 0 0 0))
@@
       (net 20 "Net-(D212-Pad2)"))
     (model Socket_Strips.3dshapes/Socket_Strip_Straight_1x03.wrl
-      (at (xyz 0.1 0 0))
+      (offset (xyz 2.539999961853027 0 0))
       (scale (xyz 1 1 1))
       (rotate (xyz 0 0 180))
@@
     (pad 1 thru_hole circle (at 0 0) (size 6.4 6.4) (drill 3.2) (layers *.Cu *.Mask))
   )
-  (gr_text "MM6D    2020" (at 163.068 124.46) (layer B.Cu)
+  (gr_text "MM6D    2023" (at 163.068 124.46) (layer B.Cu)
     (effects (font (size 1.5 1.5) (thickness 0.3)) (justify mirror))
   )
-  (gr_text "DN: 59/11/5" (at 163.576 124.46) (layer F.SilkS)
-    (effects (font (size 1.5 1.5) (thickness 0.3)))
-  )
   (gr_text "Battery\n6F22" (at 165.608 69.088) (layer F.SilkS)
