File: cad_files/display/display.sch (KiCad schematic (older format))
At the start: 34 parts, among them P106 CONN_01X02, SW1a1 auxcontalt, SW1b1 auxcontalt, SW2a1 auxcontalt, SW2b1 auxcontalt, SW3a1 auxcontalt, SW3b1 auxcontalt, SW4 auxcontalt

Commit message: 201026
Parts:
- removed P? (x2): CONN_01X01, symbol CONN_01X01
- removed SW1a1, SW1b1, SW2a1, SW2b1, SW3a1, SW3b1, SW4: auxcontalt, symbol auxcontalt
- added P202, P208, P209: CONN_01X01, Socket_Strips:Socket_Strip_Straight_1x01, symbol CONN_01X01
- added P206, P207: CONN_01X03, Socket_Strips:Socket_Strip_Straight_1x03, symbol CONN_01X03
- BT201: renamed from BT2; footprint (none) -> Socket_Strips:Socket_Strip_Straight_1x02; Field4 6F22 battery -> 6F22
- D201: renamed from D1; footprint (none) -> LEDs:LED-5MM
- D202: renamed from D2; footprint (none) -> LEDs:LED-5MM
- D203: renamed from D3; footprint (none) -> LEDs:LED-5MM
- D204: renamed from D4; footprint (none) -> LEDs:LED-5MM
- D205: renamed from D5; footprint (none) -> LEDs:LED-5MM
- D206: renamed from D6; footprint (none) -> LEDs:LED-5MM
- D207: renamed from D7; footprint (none) -> LEDs:LED-5MM
- D208: renamed from D8; footprint (none) -> LEDs:LED-5MM
- D209: renamed from D9; footprint (none) -> LEDs:LED-5MM
- D210: renamed from D11; footprint (none) -> Diodes_THT:Diode_DO-41_SOD81_Horizontal_RM10
- D211: renamed from D10; footprint (none) -> Diodes_THT:Diode_DO-41_SOD81_Horizontal_RM10
- D212: renamed from D12; footprint (none) -> Diodes_THT:Diode_DO-41_SOD81_Horizontal_RM10
- P201: renamed from P106; footprint (none) -> Socket_Strips:Socket_Strip_Straight_1x02
- P203: renamed from P?; footprint (none) -> Socket_Strips:Socket_Strip_Straight_1x01
- P204: renamed from P?; footprint (none) -> Socket_Strips:Socket_Strip_Straight_1x06
- P205: renamed from P?; footprint (none) -> Socket_Strips:Socket_Strip_Straight_1x02
- R201: renamed from R1; footprint (none) -> Resistors_THT:Resistor_Horizontal_RM15mm
- R202: renamed from R2; footprint (none) -> Resistors_THT:Resistor_Horizontal_RM15mm
- R203: renamed from R3; footprint (none) -> Resistors_THT:Resistor_Horizontal_RM15mm
- R204: renamed from R4; footprint (none) -> Resistors_THT:Resistor_Horizontal_RM15mm
- R205: renamed from R5; footprint (none) -> Resistors_THT:Resistor_Horizontal_RM15mm
- R206: renamed from R6; footprint (none) -> Resistors_THT:Resistor_Horizontal_RM15mm
- R207: renamed from R7; footprint (none) -> Resistors_THT:Resistor_Horizontal_RM15mm
- R208: renamed from R8; footprint (none) -> Resistors_THT:Resistor_Horizontal_RM15mm
Connections:
- net labels added: +12V
- net labels removed: 0V
- wire segments 73 -> 64
- no-connect marks 4 -> 0
Other:
- note added: "Alarm\nGeneral error"
- note removed: "Alarm\nError"
- note removed: "Manual\n mode"
- note removed: "Operation\n mode"
- note removed: "front panel"
- moved on the sheet: BT201, D201, D202, D203, D204, D205, D206, D207, D208, D209, D210, D211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

Commit message: 201026
Parts:
- removed P205: CONN_01X02, Socket_Strips:Socket_Strip_Straight_1x02, symbol CONN_01X02
- added P205: CONN_01X03, Socket_Strips:Socket_Strip_Straight_1x03, symbol CONN_01X03
Connections:
- net at D212.2 (A): now also P205.1 (P1)
- net at D201.1 (K): now also P205.3 (P3)
- net at P201.1 (P1): now also D209.2 (A); no longer D209.1 (K)
- net at P201.2 (P2): now also D209.1 (K); no longer D209.2 (A)
Changed lines of the file:
@@
 F 3 "" H 3625 1850 50  0000 C CNN
 	1    3625 1850
-	0    -1   -1   0
+	0    1    -1   0
 $EndComp
 $Comp
@@
 	6425 2500 6525 2500
 $Comp
-L CONN_01X02 P205
-U 1 1 5F95DF9F
-P 6475 1850
-F 0 "P205" V 6600 1825 50  0000 C CNN
-F 1 "CONN_01X02" V 6575 1850 50  0001 C CNN
-F 2 "Socket_Strips:Socket_Strip_Straight_1x02" H 6475 1850 50  0001 C CNN
-F 3 "" H 6475 1850 50  0000 C CNN
-	1    6475 1850
-	0    -1   -1   0
-$EndComp
-$Comp
 L CONN_01X06 P204
 U 1 1 5F95E0A1
@@
 	4950 2500 4950 2275
 Wire Wire Line
-	4950 2275 6425 2275
-Wire Wire Line
-	6425 2275 6425 2050
+	4950 2275 6325 2275
 $Comp
 L CONN_01X03 P206
@@
 	6775 2050 6775 5275
 Wire Wire Line
-	4225 5025 4225 3050
+	4225 3050 4225 5025
 Wire Wire Line
 	7425 5525 5925 5525
@@
 Wire Wire Line
 	7425 2050 7425 5525
+$Comp
+L CONN_01X03 P205
+U 1 1 5F96B4A5
+P 6425 1850
+F 0 "P205" V 6550 1850 50  0000 C CNN
+F 1 "CONN_01X03" V 6525 1850 50  0001 C CNN
+F 2 "Socket_Strips:Socket_Strip_Straight_1x03" H 6425 1850 50  0001 C CNN
+F 3 "" H 6425 1850 50  0000 C CNN
+	1    6425 1850
+	0    1    -1   0
+$EndComp
+Wire Wire Line
+	6325 2275 6325 2050
 $EndSCHEMATC

Commit message: 201029
Connections:
- net at D212.2 (A): now also P205.3 (P3); no longer P205.1 (P1)
- net at D201.1 (K): now also P205.1 (P1); no longer P205.3 (P3)
- net at P201.1 (P1): now also D209.1 (K); no longer D209.2 (A)
- net at P201.2 (P2): now also D209.2 (A); no longer D209.1 (K)
Changed lines of the file:
@@
 F 3 "" H 3625 1850 50  0000 C CNN
 	1    3625 1850
-	0    1    -1   0
+	0    -1   -1   0
 $EndComp
 $Comp
@@
 F 3 "" H 6425 1850 50  0000 C CNN
 	1    6425 1850
-	0    1    -1   0
-$EndComp
-Wire Wire Line
+	0    -1   -1   0
+$EndComp
+Wire Wire Line

Commit message: 201226
Parts:
- R201: value 47k -> 220k
- R202, R203: value 1.5k -> 9.1k
- R204, R205, R206, R207, R208: value 1,5k -> 9.1k
Changed lines of the file:
@@
 P 5850 2500
 F 0 "R201" V 5750 2500 50  0000 C CNN
-F 1 "47k" V 5950 2500 50  0000 C CNN
+F 1 "220k" V 5950 2500 50  0000 C CNN
 F 2 "Resistors_THT:Resistor_Horizontal_RM15mm" V 5780 2500 50  0001 C CNN
 F 3 "" H 5850 2500 50  0000 C CNN
@@
 P 5250 2500
 F 0 "D201" H 5525 2550 50  0000 C CNN
-F 1 "white" H 5475 2450 50  0000 C CNN
+F 1 "white" H 5525 2450 50  0000 C CNN
 F 2 "LEDs:LED-5MM" H 5250 2500 50  0001 C CNN
 F 3 "" H 5250 2500 50  0000 C CNN
@@
 P 5875 4425
 F 0 "R208" V 5775 4425 50  0000 C CNN
-F 1 "1,5k" V 5975 4425 50  0000 C CNN
+F 1 "9.1k" V 5975 4425 50  0000 C CNN
 F 2 "Resistors_THT:Resistor_Horizontal_RM15mm" V 5805 4425 50  0001 C CNN
 F 3 "" H 5875 4425 50  0000 C CNN
@@
 P 5250 4150
 F 0 "D207" H 5525 4200 50  0000 C CNN
-F 1 "red" H 5525 4100 50  0000 C CNN
+F 1 "red" H 5500 4100 50  0000 C CNN
 F 2 "LEDs:LED-5MM" H 5250 4150 50  0001 C CNN
 F 3 "" H 5250 4150 50  0000 C CNN
@@
 P 5875 3050
 F 0 "R203" V 5775 3050 50  0000 C CNN
-F 1 "1.5k" V 5975 3050 50  0000 C CNN
+F 1 "9.1k" V 5975 3050 50  0000 C CNN
 F 2 "Resistors_THT:Resistor_Horizontal_RM15mm" V 5805 3050 50  0001 C CNN
 F 3 "" H 5875 3050 50  0000 C CNN
@@
 P 5250 3050
 F 0 "D203" H 5525 3100 50  0000 C CNN
-F 1 "white" H 5475 3000 50  0000 C CNN
+F 1 "white" H 5525 3000 50  0000 C CNN
 F 2 "LEDs:LED-5MM" H 5250 3050 50  0001 C CNN
 F 3 "" H 5250 3050 50  0000 C CNN
@@
 P 5875 4150
 F 0 "R207" V 5800 4150 50  0000 C CNN
-F 1 "1,5k" V 5975 4150 50  0000 C CNN
+F 1 "9.1k" V 5975 4150 50  0000 C CNN
 F 2 "Resistors_THT:Resistor_Horizontal_RM15mm" V 5805 4150 50  0001 C CNN
 F 3 "" H 5875 4150 50  0000 C CNN
@@
 P 5250 4425
 F 0 "D208" H 5525 4475 50  0000 C CNN
-F 1 "yellow" H 5475 4375 50  0000 C CNN
+F 1 "yellow" H 5550 4375 50  0000 C CNN
 F 2 "LEDs:LED-5MM" H 5250 4425 50  0001 C CNN
 F 3 "" H 5250 4425 50  0000 C CNN
@@
 P 5875 3875
 F 0 "R206" V 5800 3875 50  0000 C CNN
-F 1 "1,5k" V 5975 3875 50  0000 C CNN
+F 1 "9.1k" V 5975 3875 50  0000 C CNN
 F 2 "Resistors_THT:Resistor_Horizontal_RM15mm" V 5805 3875 50  0001 C CNN
 F 3 "" H 5875 3875 50  0000 C CNN
@@
 P 5250 3875
 F 0 "D206" H 5525 3925 50  0000 C CNN
-F 1 "green" H 5475 3825 50  0000 C CNN
+F 1 "green" H 5525 3825 50  0000 C CNN
 F 2 "LEDs:LED-5MM" H 5250 3875 50  0001 C CNN
 F 3 "" H 5250 3875 50  0000 C CNN
@@
 P 5875 3600
 F 0 "R205" V 5800 3600 50  0000 C CNN
-F 1 "1,5k" V 5975 3600 50  0000 C CNN
+F 1 "9.1k" V 5975 3600 50  0000 C CNN
 F 2 "Resistors_THT:Resistor_Horizontal_RM15mm" V 5805 3600 50  0001 C CNN
 F 3 "" H 5875 3600 50  0000 C CNN
@@
 P 5250 3600
 F 0 "D205" H 5525 3650 50  0000 C CNN
-F 1 "green" H 5475 3550 50  0000 C CNN
+F 1 "green" H 5525 3550 50  0000 C CNN
 F 2 "LEDs:LED-5MM" H 5250 3600 50  0001 C CNN
 F 3 "" H 5250 3600 50  0000 C CNN
@@
 P 5875 3325
 F 0 "R204" V 5800 3325 50  0000 C CNN
-F 1 "1,5k" V 5975 3325 50  0000 C CNN
+F 1 "9.1k" V 5975 3325 50  0000 C CNN
 F 2 "Resistors_THT:Resistor_Horizontal_RM15mm" V 5805 3325 50  0001 C CNN
 F 3 "" H 5875 3325 50  0000 C CNN
@@
 P 5250 3325
 F 0 "D204" H 5525 3375 50  0000 C CNN
-F 1 "green" H 5475 3275 50  0000 C CNN
+F 1 "green" H 5525 3275 50  0000 C CNN
 F 2 "LEDs:LED-5MM" H 5250 3325 50  0001 C CNN
 F 3 "" H 5250 3325 50  0000 C CNN
@@
 P 5850 2775
 F 0 "R202" V 5750 2775 50  0000 C CNN
-F 1 "1.5k" V 5950 2775 50  0000 C CNN
+F 1 "9.1k" V 5950 2775 50  0000 C CNN
 F 2 "Resistors_THT:Resistor_Horizontal_RM15mm" V 5780 2775 50  0001 C CNN
 F 3 "" H 5850 2775 50  0000 C CNN

Commit message: 240423
Parts:
- BT201: symbol Battery -> display-rescue:Battery
- D201, D202, D203, D204, D205, D206, D207, D208, D209: symbol LED-CIRCLE -> pzs_devices:LED-CIRCLE
- D210, D211, D212: symbol D -> display-rescue:D
- P201: symbol CONN_01X02 -> display-rescue:CONN_01X02
- P202, P203, P208, P209: symbol CONN_01X01 -> display-rescue:CONN_01X01
- P204: symbol CONN_01X06 -> display-rescue:CONN_01X06
- P205, P206, P207: symbol CONN_01X03 -> display-rescue:CONN_01X03
- R201, R202, R203, R204, R205, R206, R207, R208: symbol R -> display-rescue:R
Changed lines of the file:
@@
-EESchema Schematic File Version 2
-LIBS:pzs_others
-LIBS:power
-LIBS:device
-LIBS:transistors
-LIBS:conn
-LIBS:linear
-LIBS:regul
-LIBS:74xx
-LIBS:cmos4000
-LIBS:adc-dac
-LIBS:memory
-LIBS:xilinx
-LIBS:microcontrollers
-LIBS:dsp
-LIBS:microchip
-LIBS:analog_switches
-LIBS:motorola
-LIBS:texas
-LIBS:intel
-LIBS:audio
-LIBS:interface
-LIBS:digital-audio
-LIBS:philips
-LIBS:display
-LIBS:cypress
-LIBS:siliconi
-LIBS:opto
-LIBS:atmel
-LIBS:contrib
-LIBS:valves
-LIBS:pzs_devices
-LIBS:display-cache
-EELAYER 25 0
+EESchema Schematic File Version 4
+EELAYER 30 0
 EELAYER END
 $Descr A4 11693 8268
 encoding utf-8
 Sheet 1 1
-Title "MM6D Remote controlled switching device"
-Date "2020-06-12"
-Rev "200612"
-Comp "Pozsar Zsolt - http://www.szerafingomba.hu"
+Title "MM6D Grow house control device"
+Date "2024-04-23"
+Rev "231006"
+Comp "Pozsar Zsolt - http://www.pozsarzs.hu"
 Comment1 "Display board"
 Comment2 ""
 Comment3 ""
-Comment4 "Draw no.: 59/11/4"
+Comment4 ""
 $EndDescr
 $Comp
-L R R201
+L display-rescue:R R201
 U 1 1 5F1AEEAF
 P 5850 2500
@@
 $EndComp
 $Comp
-L D D212
+L display-rescue:D D212
 U 1 1 5F1AEFFD
 P 6275 2500
@@
 $EndComp
 $Comp
-L LED-CIRCLE D201
+L pzs_devices:LED-CIRCLE D201
 U 1 1 5F1AF03C
 P 5250 2500
@@
 $EndComp
 $Comp
-L R R208
+L display-rescue:R R208
 U 1 1 5F1BBBB6
 P 5875 4425
@@
 $EndComp
 $Comp
-L LED-CIRCLE D207
+L pzs_devices:LED-CIRCLE D207
 U 1 1 5F1BBBBC
 P 5250 4150
@@
 Protection\nerror
 $Comp
-L R R203
+L display-rescue:R R203
 U 1 1 5F1C190A
 P 5875 3050
@@
 $EndComp
 $Comp
-L LED-CIRCLE D203
+L pzs_devices:LED-CIRCLE D203
 U 1 1 5F1C1910
 P 5250 3050
@@
 Auxiliary\nvoltage
 $Comp
-L R R207
+L display-rescue:R R207
 U 1 1 5F1C6BF7
 P 5875 4150
@@
 $EndComp
 $Comp
-L LED-CIRCLE D208
+L pzs_devices:LED-CIRCLE D208
 U 1 1 5F1C6BFD
 P 5250 4425
@@
 Manual\nmode
 $Comp
-L D D210
+L display-rescue:D D210
 U 1 1 5F1CC812
 P 5325 5275
@@
 $EndComp
 $Comp
-L D D211
+L display-rescue:D D211
 U 1 1 5F1CC947
 P 5325 5525
@@
 $EndComp
 $Comp
-L Battery BT201
+L display-rescue:Battery BT201
 U 1 1 5F1CCA80
 P 5725 5525
@@
 $EndComp
 $Comp
-L CONN_01X02 P201
+L display-rescue:CONN_01X02 P201
 U 1 1 5F81A1FB
 P 3625 1850
@@
 $EndComp
 $Comp
-L LED-CIRCLE D209
+L pzs_devices:LED-CIRCLE D209
 U 1 1 5F81AC4E
 P 5250 4750
@@
 Active
 $Comp
-L R R206
+L display-rescue:R R206
 U 1 1 5F7E9A89
 P 5875 3875
@@
 $EndComp
 $Comp
-L LED-CIRCLE D206
+L pzs_devices:LED-CIRCLE D206
 U 1 1 5F7E9A8F
 P 5250 3875
@@
 $EndComp
 $Comp
-L R R205
+L display-rescue:R R205
 U 1 1 5F7E9BE3
 P 5875 3600
@@
 $EndComp
 $Comp
-L LED-CIRCLE D205
+L pzs_devices:LED-CIRCLE D205
 U 1 1 5F7E9BE9
 P 5250 3600
@@
 $EndComp
 $Comp
-L R R204
+L display-rescue:R R204
 U 1 1 5F7E9D3D
 P 5875 3325
@@
 $EndComp
 $Comp
-L LED-CIRCLE D204
+L pzs_devices:LED-CIRCLE D204
 U 1 1 5F7E9D43
 P 5250 3325
@@
 	5075 5525 5075 5275
 Wire Wire Line
-	3925 5275 5175 5275
+	3925 5275 5075 5275
 Wire Wire Line
 	6775 5275 5475 5275
@@
 Connection ~ 6775 3875
 $Comp
-L LED-CIRCLE D202
+L pzs_devices:LED-CIRCLE D202
 U 1 1 5F7F615E
 P 5250 2775
@@
 $EndComp
 $Comp
-L R R202
+L display-rescue:R R202
 U 1 1 5F7F6998
 P 5850 2775
@@
 	6425 2500 6525 2500
 $Comp
-L CONN_01X06 P204
+L display-rescue:CONN_01X06 P204
 U 1 1 5F95E0A1
 P 4675 1850
@@
 Lamp\non
 $Comp
-L CONN_01X01 P203
+L display-rescue:CONN_01X01 P203
 U 1 1 5F95EDE5
 P 4175 1850
@@
 $EndComp
 Wire Wire Line
-	4425 2050 4425 3325
+	4425 2050 4425 2150
 Wire Wire Line
 	4425 2150 4525 2150
@@
 	4525 2150 4525 2050
 Wire Wire Line
-	4625 2050 4625 3600
+	4625 2050 4625 2150
 Wire Wire Line
 	4625 2150 4725 2150
@@
 	4725 2150 4725 2050
 Wire Wire Line
-	4825 2050 4825 3875
+	4825 2050 4825 2150
 Wire Wire Line
 	4825 2150 4925 2150
@@
 	4950 2275 6325 2275
 $Comp
-L CONN_01X03 P206
+L display-rescue:CONN_01X03 P206
 U 1 1 5F969BAC
 P 6875 1850
@@
 $EndComp
 $Comp
-L CONN_01X03 P207
+L display-rescue:CONN_01X03 P207
 U 1 1 5F969DAF
 P 7325 1850
@@
 $EndComp
 Wire Wire Line
-	6775 2150 6975 2150
+	6775 2150 6875 2150
 Wire Wire Line
 	6975 2150 6975 2050
@@
 	7225 2050 7225 2150
 Wire Wire Line
-	7225 2150 7425 2150
+	7225 2150 7325 2150
 Wire Wire Line
 	7325 2050 7325 2150
@@
 Connection ~ 4225 4425
 $Comp
-L CONN_01X01 P208
+L display-rescue:CONN_01X01 P208
 U 1 1 5F96B08E
 P 7675 1850
@@
 $EndComp
 $Comp
-L CONN_01X01 P209
+L display-rescue:CONN_01X01 P209
 U 1 1 5F96B12A
 P 7925 1850
@@
 	7925 4425 7925 2050
 Wire Wire Line
-	6775 2050 6775 5275
-Wire Wire Line
-	4225 3050 4225 5025
+	6775 2050 6775 2150
+Wire Wire Line
+	4225 3050 4225 4150
 Wire Wire Line
 	7425 5525 5925 5525
 Connection ~ 7425 5025
 $Comp
-L CONN_01X01 P202
+L display-rescue:CONN_01X01 P202
 U 1 1 5F96D0B3
 P 3925 1850
@@
 +12V
 Wire Wire Line
-	7425 2050 7425 5525
-$Comp
-L CONN_01X03 P205
+	7425 2050 7425 2150
+$Comp
+L display-rescue:CONN_01X03 P205
 U 1 1 5F96B4A5
 P 6425 1850
@@
 Wire Wire Line
 	6325 2275 6325 2050
+Wire Wire Line
+	5075 5275 5175 5275
+Wire Wire Line
+	4225 4150 4225 4425
+Wire Wire Line
+	6775 3050 6775 3325
+Wire Wire Line
+	6775 3325 6775 3600
+Wire Wire Line
+	6775 3600 6775 3875
+Wire Wire Line
+	6775 3875 6775 5275
+Wire Wire Line
+	6775 2775 6775 3050
+Wire Wire Line
+	4425 2150 4425 3325
+Wire Wire Line
+	4625 2150 4625 3600
+Wire Wire Line
+	4825 2150 4825 3875
+Wire Wire Line
+	6875 2150 6975 2150
+Wire Wire Line
+	7325 2150 7425 2150
+Wire Wire Line
+	6775 2150 6775 2775
+Wire Wire Line
+	7425 2150 7425 5025
+Wire Wire Line
+	4225 4425 4225 5025
+Wire Wire Line
+	7425 5025 7425 5525
 $EndSCHEMATC
